Commit message: p n p, pan_tilt_mover, hector fix, gripper controller fix, dxl vel formula fix

File: armadillo2_utils/softkinetic/softkinetic_camera/urdf/sofkinetic_ds325.xacro (robot description, xacro)
@@ -5,5 +5,5 @@
     <!-- Add frames for RGB and depth optical axes -->
     <joint name="${name}_rgb_joint" type="fixed">
-      <origin xyz="0.0 0.0125 0.0" rpy="0.0 0.0 0.0"/>
+      <origin xyz="0.02 -0.0125 0.0" rpy="0.0 0.0 0.0"/>
       <parent link="${name}_link"/>
       <child link="${name}_rgb_frame"/>
@@ -17,5 +17,5 @@
     <link name="${name}_rgb_optical_frame"/>
     <joint name="${name}_depth_joint" type="fixed">
-      <origin xyz="0.0 -0.0125 0.0" rpy="0.0 0.0 0.0"/>
+      <origin xyz="0.0 0.0125 0.0" rpy="0.0 0.0 0.0"/>
       <parent link="${name}_link"/>
       <child link="${name}_depth_frame"/>
