Commit message: gazebo imu and gps plugins

File: armadillo2_description/urdf/armadillo2_gazebo.xacro (robot description, xacro)
@@ -39,13 +39,10 @@
   <xacro:if value="$(arg gps)">
     <xacro:include filename="$(find armadillo2_gazebo)/macros/gps.xacro" />
-    <xacro:gps />
+    <xacro:gps link="base_link" hz="5" topic="GPS" lat="31.262218" long="34.80146100" alt="298"/>
   </xacro:if>
   <!-- IMU   -->
   <xacro:if value="$(arg imu)">
     <xacro:include filename="$(find armadillo2_gazebo)/macros/imu.xacro" />
-    <xacro:imu link="base_link" imu_offset_x="0" imu_offset_y="0" imu_offset_z="${M_PI}"
-      imu_offset_roll="0" imu_offset_pitch="0"
-      imu_offset_yaw="0" mag_offset_x="0"
-      mag_offset_y="0" mag_offset_z="0" />
+    <xacro:imu link="base_link" hz="50" topic="IMU" />
     </xacro:if>
 <gazebo>

File: armadillo2_gazebo/macros/gps.xacro (robot description, xacro)
@@ -1,14 +1,18 @@
+<?xml version="1.0"?>
 <robot xmlns:xacro="http://www.ros.org/wiki/xacro" name="GPS" description="GPS sensor">
-	<xacro:macro name="gps" >
+<xacro:macro name="gps" params="link hz topic lat long alt">
 		<gazebo>
 			<plugin name="GazeboRosGps" filename="libhector_gazebo_ros_gps.so">
-				<updateRate>50.0</updateRate>
-				<bodyName>base_link</bodyName>
-				<frameId>base_link</frameId>
-				<topicName>GPS/fix</topicName>
+				<updateRate>${hz}</updateRate>
+				<bodyName>${link}</bodyName>
+				<frameId>${link}</frameId>
+				<topicName>${topic}/fix</topicName>
 				<serviceName>SERVICE_GPS</serviceName>
-				<velocityTopicName>GPS/fix_velocity</velocityTopicName>
+				<velocityTopicName>${topic}/fix_velocity</velocityTopicName>
 				<gaussianNoise>2.89e-08 2.89e-08 2.89e-08</gaussianNoise>
 				<velocityGaussianNoise>2.89e-08 2.89e-08 2.89e-08</velocityGaussianNoise>
+				<referenceLatitude>${lat}</referenceLatitude>
+				<referenceLongitude>${long}</referenceLongitude>
+				<referenceAltitude>${alt}</referenceAltitude>
 			</plugin>
 		</gazebo>

File: armadillo2_gazebo/macros/imu.xacro (robot description, xacro)
@@ -1,33 +1,24 @@
+<?xml version="1.0"?>
 <robot xmlns:xacro="http://www.ros.org/wiki/xacro" name="IMU" description="IMU sensor">
-	<xacro:macro name="imu" params="link imu_offset_x imu_offset_y imu_offset_z imu_offset_roll imu_offset_pitch imu_offset_yaw mag_offset_x mag_offset_y mag_offset_z">
-		<gazebo>
-			<plugin name="GazeboRosImu" filename="libhector_gazebo_ros_imu.so">
-				<alwaysOn>true</alwaysOn>
-				<updateRate>50.0</updateRate>
-				<bodyName>${link}</bodyName>
-				<frameId>${link}</frameId>
-				<topicName>imu</topicName>
-<accelDrift>0.001 0.001 0.001</accelDrift>
-      <accelGaussianNoise>0.05 0.05 0.05</accelGaussianNoise>
-      <rateDrift>0.005 0.005 0.005 </rateDrift>
-      <rateGaussianNoise>0.005 0.005 0.005 </rateGaussianNoise>
-      <headingDrift>0.005</headingDrift>
-      <headingGaussianNoise>0.005</headingGaussianNoise>
-				<xyzOffsets>${imu_offset_x} ${imu_offset_y} ${imu_offset_z}</xyzOffsets>
-				<rpyOffsets>${imu_offset_roll} ${imu_offset_pitch} ${imu_offset_yaw}</rpyOffsets>
-				<material>Gazebo/Red</material>
-			</plugin>
-		</gazebo>
-		<gazebo>
-			<plugin name="GazeboRosMagnetic" filename="libhector_gazebo_ros_magnetic.so">
-				<updateRate>50.0</updateRate>
-				<bodyName>${link}</bodyName>
-				<frameId>${link}</frameId>
-				<topicName>imu_M</topicName>
-				<offset>${mag_offset_x} ${mag_offset_y} ${mag_offset_z}</offset>
-				<drift>0.0 0.0 0.0</drift>
-				<gaussianNoise>1.3e-2 1.3e-2 1.3e-2</gaussianNoise>
-			</plugin>
-		</gazebo>
+	<xacro:macro name="imu" params="link hz topic">
+ <gazebo reference="${link}">
+    <gravity>true</gravity>
+    <sensor name="imu_sensor" type="imu">
+      <always_on>true</always_on>
+      <update_rate>${hz}</update_rate>
+      <visualize>true</visualize>
+      <topic>__default_topic__</topic>
+      <plugin filename="libgazebo_ros_imu_sensor.so" name="imu_plugin">
+        <topicName>${topic}</topicName>
+        <bodyName>${link}</bodyName>
+        <updateRateHZ>10.0</updateRateHZ>
+        <gaussianNoise>0.0</gaussianNoise>
+        <xyzOffset>0 0 0</xyzOffset>
+        <rpyOffset>0 0 0</rpyOffset>
+        <frameName>${link}</frameName>
+      </plugin>
+      <pose>0 0 0 0 0 0</pose>
+    </sensor>
+  </gazebo>
 	</xacro:macro>
 </robot>

Commit message: gazebo urf plugin

File: armadillo2_description/urdf/armadillo2_gazebo.xacro (robot description, xacro)
@@ -29,5 +29,5 @@
   <xacro:if value="$(arg urf)">
     <xacro:include filename="$(find armadillo2_gazebo)/macros/urf.xacro" />
-    <xacro:urf name="rear" link="front_urf_link" topic="URF/front" />
+    <xacro:urf name="front" link="front_urf_link" topic="URF/front" fov="${5.0*M_PI/180}" min="0.2" max="5.0"/>
   </xacro:if>
   <!-- hokuyo   -->

File: armadillo2_gazebo/macros/urf.xacro (robot description, xacro)
@@ -1,4 +1,4 @@
 <robot xmlns:xacro="http://www.ros.org/wiki/xacro" name="URF" description="URF sensor">
- 	<xacro:macro name="urf" params=" name link topic">
+ 	<xacro:macro name="urf" params=" name link topic fov min max">
 		<gazebo reference="${link}">
 			<material>Gazebo/Black</material>
@@ -13,17 +13,17 @@
 							<samples>10</samples>
 							<resolution>1</resolution>
-							<min_angle>${-URF_FOV/2.0}</min_angle>
-							<max_angle>${URF_FOV/2.0}</max_angle>
+							<min_angle>${-fov/2.0}</min_angle>
+							<max_angle>${-fov/2.0}</max_angle>
 						</horizontal>
 						<vertical>
 							<samples>10</samples>
 							<resolution>1</resolution>
-							<min_angle>${-URF_FOV/2.0}</min_angle>
-							<max_angle>${URF_FOV/2.0}</max_angle>
+							<min_angle>${-fov/2.0}</min_angle>
+							<max_angle>${-fov/2.0}</max_angle>
 						</vertical>
 					</scan>
 					<range>
-						<min>0.01</min>
-						<max>5.0</max>
+						<min>${min}</min>
+						<max>${max}</max>
 						<resolution>0.001</resolution>
 					</range>

Commit message: urf gazebo plugin fix fov

File: armadillo2_description/urdf/armadillo2_gazebo.xacro (robot description, xacro)
@@ -3,5 +3,4 @@
  <xacro:include filename="$(find armadillo2_description)/urdf/armadillo2.xacro" />
 <xacro:include filename="$(find armadillo2_gazebo)/macros/softkinetic_camera_ds325.xacro" />
-  <xacro:property name="URF_FOV" value="${10.0*M_PI/180}" />
   <xacro:arg name="kinect2" default="true"/>
   <xacro:arg name="kinect2_hz" default="30.0"/>
@@ -29,5 +28,5 @@
   <xacro:if value="$(arg urf)">
     <xacro:include filename="$(find armadillo2_gazebo)/macros/urf.xacro" />
-    <xacro:urf name="front" link="front_urf_link" topic="URF/front" fov="${5.0*M_PI/180}" min="0.2" max="5.0"/>
+    <xacro:urf name="front" link="front_urf_link" topic="URF/front" fov="${10.0*M_PI/180.0}" min="0.2" max="5.0"/>
   </xacro:if>
   <!-- hokuyo  utm-30lx -->

File: armadillo2_gazebo/macros/urf.xacro (robot description, xacro)
@@ -14,5 +14,5 @@
 							<resolution>1</resolution>
 							<min_angle>${-fov/2.0}</min_angle>
-							<max_angle>${-fov/2.0}</max_angle>
+							<max_angle>${fov/2.0}</max_angle>
 						</horizontal>
 						<vertical>
@@ -20,5 +20,5 @@
 							<resolution>1</resolution>
 							<min_angle>${-fov/2.0}</min_angle>
-							<max_angle>${-fov/2.0}</max_angle>
+							<max_angle>${fov/2.0}</max_angle>
 						</vertical>
 					</scan>
