Commit message: controllers

File: armadillo2_description/urdf/armadillo2.xacro (robot description, xacro)
@@ -1,4 +1,4 @@
 <?xml version="1.0"?>
-<robot xmlns:xacro="http://www.ros.org/wiki/xacro" name="armadillo_robot" description="ARMadillo Robot">
+<robot xmlns:xacro="http://www.ros.org/wiki/xacro" name="armadillo2_robot" description="ARMadillo Robot">
  <xacro:property name="M_PI" value="3.1415926535897931" />
 <link name="base_footprint"/>
@@ -15,7 +15,7 @@
         rpy="0 0 0" />
       <mass
-        value="80.6774" />
-      <inertia
-        ixx="0.61071"
+        value="1.6774" />
+      <inertia
+        ixx="50.61071"
         ixy="2.5604E-05"
         ixz="-0.080403"
@@ -131,5 +131,6 @@
         rpy="${M_PI/2} 0 0" />
       <geometry>
-      <cylinder  length="0.04" radius="0.1"/>
+      <cylinder  length="0.04" radius="0.12"/>
+<!--        0.1 ********************************************************************************-->
       </geometry>
     </collision>
@@ -183,5 +184,6 @@
         rpy="${M_PI/2} 0 0" />
       <geometry>
-      <cylinder  length="0.04" radius="0.1"/>
+      <cylinder  length="0.04" radius="0.12"/>
+      <!--        0.1 ********************************************************************************-->
       </geometry>
     </collision>

File: armadillo2_description/urdf/armadillo2_gazebo.xacro (robot description, xacro)
@@ -1,10 +1,10 @@
 <?xml version="1.0"?>
-<robot xmlns:xacro="http://www.ros.org/wiki/xacro" name="armadillo2_robot">
+<robot xmlns:xacro="http://www.ros.org/wiki/xacro" name="armadillo_robot" description="ARMadillo Robot">
  <xacro:include filename="$(find armadillo2_description)/urdf/armadillo2.xacro" />
-        <gazebo>
+<gazebo>
             <plugin name="gazebo_ros_control" filename="libgazebo_ros_control.so">
             <robotSimType>gazebo_ros_control/Armadillo2RobotHWSim</robotSimType>
             </plugin>
-        </gazebo>
+          </gazebo>
           <transmission name="left_wheel_joint_trans">
             <type>transmission_interface/SimpleTransmission</type>

Commit message: dxl read rate

File: armadillo2_description/urdf/armadillo2.xacro (robot description, xacro)
@@ -15,5 +15,5 @@
         rpy="0 0 0" />
       <mass
-        value="1.6774" />
+        value="50.6774" />
       <inertia
         ixx="50.61071"
@@ -131,6 +131,5 @@
         rpy="${M_PI/2} 0 0" />
       <geometry>
-      <cylinder  length="0.04" radius="0.12"/>
-<!--        0.1 ********************************************************************************-->
+      <cylinder  length="0.04" radius="0.1"/>
       </geometry>
     </collision>
@@ -184,6 +183,5 @@
         rpy="${M_PI/2} 0 0" />
       <geometry>
-      <cylinder  length="0.04" radius="0.12"/>
-      <!--        0.1 ********************************************************************************-->
+      <cylinder  length="0.04" radius="0.1"/>
       </geometry>
     </collision>

Commit message: softkinetic --tested ok

File: armadillo2_description/urdf/armadillo2.xacro (robot description, xacro)
@@ -2,4 +2,5 @@
 <robot xmlns:xacro="http://www.ros.org/wiki/xacro" name="armadillo2_robot" description="ARMadillo Robot">
  <xacro:property name="M_PI" value="3.1415926535897931" />
+ <xacro:include filename="$(find softkinetic_camera)/urdf/sofkinetic_ds325.xacro"/>
 <link name="base_footprint"/>
  <joint name="base_footprint_joint" type="fixed">
@@ -948,5 +949,5 @@
   </joint>
   <link
-    name="softkinetic_link">
+    name="softkinetic_camera_link">
     <inertial>
       <origin
@@ -996,37 +997,10 @@
       link="wrist_link" />
     <child
-      link="softkinetic_link" />
+      link="softkinetic_camera_link" />
     <axis
       xyz="0 0 0" />
   </joint>
-  <link
-    name="softkinetic_left_link" />
-  <joint
-    name="softkinetic_left_joint"
-    type="fixed">
-    <origin
-      xyz="0.0083 0.0135 0"
-      rpy="0 0 0" />
-    <parent
-      link="softkinetic_link" />
-    <child
-      link="softkinetic_left_link" />
-    <axis
-      xyz="0 0 0" />
-  </joint>
-  <link
-    name="softkinetic_right_link" />
-  <joint
-    name="softkinetic_right_joint"
-    type="fixed">
-    <origin
-      xyz="0.0083 -0.0135 0"
-      rpy="-8.0779E-28 0 1.3535E-11" />
-    <parent
-      link="softkinetic_link" />
-    <child
-      link="softkinetic_right_link" />
-    <axis
-      xyz="0 0 0" />
-  </joint>
+<softkinetic_camera name="softkinetic_camera" >
+    <origin xyz="-0.05905 0 0.0753" rpy="0.0 -${M_PI/2} 0.0"/>
+</softkinetic_camera>
 </robot>

Commit message: fixing reading delay b/w ric and pc

File: armadillo2_description/urdf/armadillo2.xacro (robot description, xacro)
@@ -464,7 +464,7 @@
   </joint>
   <link
-    name="kineckt_link" />
-  <joint
-    name="kineckt_joint"
+    name="kinect2_link" />
+  <joint
+    name="kinect2_joint"
     type="fixed">
     <origin
@@ -474,8 +474,64 @@
       link="head_tilt_link" />
     <child
-      link="kineckt_link" />
+      link="kinect2_link" />
     <axis
       xyz="0 0 0" />
   </joint>
+   <joint name="kinect2_rgb_joint" type="fixed">
+      <origin xyz="0 -0.0935 0" rpy="0 0 0"/>
+      <parent link="kinect2_link"/>
+      <child link="kinect2_rgb_frame" />
+    </joint>
+    <link name="kinect2_rgb_frame">
+      <inertial>
+	<mass value="0.001" />
+	<origin xyz="0 0 0" />
+	<inertia ixx="0.0001" ixy="0.0" ixz="0.0"
+	  iyy="0.0001" iyz="0.0"
+	  izz="0.0001" />
+	</inertial>
+      </link>
+      <joint name="kinect2_rgb_optical_joint" type="fixed">
+	<origin xyz="0 0 0" rpy="${-M_PI/2} 0 ${-M_PI/2}" />
+	<parent link="kinect2_rgb_frame" />
+	<child link="kinect2_rgb_optical_frame" />
+      </joint>
+      <link name="kinect2_rgb_optical_frame">
+	<inertial>
+	  <mass value="0.001" />
+	  <origin xyz="0 0 0" />
+	  <inertia ixx="0.0001" ixy="0.0" ixz="0.0"
+	    iyy="0.0001" iyz="0.0"
+	    izz="0.0001" />
+	  </inertial>
+	</link>
+	<joint name="kinect2_depth_joint" type="fixed">
+	  <origin xyz="0 0 0" rpy="0 0 0" />
+	  <parent link="kinect2_rgb_frame" />
+	  <child link="kinect2_depth_frame" />
+	</joint>
+	<link name="kinect2_depth_frame">
+	  <inertial>
+	    <mass value="0.001" />
+	    <origin xyz="0 0 0" />
+	    <inertia ixx="0.0001" ixy="0.0" ixz="0.0"
+	      iyy="0.0001" iyz="0.0"
+	      izz="0.0001" />
+	    </inertial>
+	  </link>
+	  <joint name="kinect2_depth_optical_joint" type="fixed">
+	    <origin xyz="0 0 0" rpy="${-M_PI/2} 0 ${-M_PI/2}" />
+	    <parent link="kinect2_depth_frame" />
+	    <child link="kinect2_depth_optical_frame" />
+	  </joint>
+	  <link name="kinect2_depth_optical_frame">
+	    <inertial>
+	      <mass value="0.001" />
+	      <origin xyz="0 0 0" />
+	      <inertia ixx="0.0001" ixy="0.0" ixz="0.0"
+		iyy="0.0001" iyz="0.0"
+		izz="0.0001" />
+	      </inertial>
+</link>
   <link
     name="rotation1_link">
