Commit message: alot!

File: armadillo2_description/urdf/armadillo2.xacro (robot description, xacro)
@@ -1,4 +1,4 @@
 <?xml version="1.0"?>
-<robot xmlns:xacro="http://www.ros.org/wiki/xacro" name="armadillo2_robot" description="ARMadillo Robot">
+<robot xmlns:xacro="http://www.ros.org/wiki/xacro" name="armadillo2_robot" description="ARMadillo2 Robot">
  <xacro:property name="M_PI" value="3.1415926535897931" />
  <xacro:include filename="$(find softkinetic_camera)/urdf/sofkinetic_ds325.xacro"/>
@@ -15,13 +15,12 @@
         xyz="-0.012353 0.000122 0.17716"
         rpy="0 0 0" />
-      <mass
-        value="50.6774" />
-      <inertia
-        ixx="50.61071"
-        ixy="2.5604E-05"
-        ixz="-0.080403"
-        iyy="0.58359"
-        iyz="-0.00032953"
-        izz="0.35309" />
+       <mass value="30.65"/>
+       <inertia
+        ixx="0.61639"
+        ixy="-9.1727E-05"
+        ixz="-0.093044"
+        iyy="0.57997"
+        iyz="5.3231E-05"
+        izz="0.36693" />
     </inertial>
     <visual>
@@ -48,22 +47,171 @@
       </geometry>
           </collision>
-      <collision name='caster_collision'>
-      <origin
-        xyz="-0.3 0 -0.0385"
-        rpy="0 0 0" />
-            <geometry>
-              <sphere radius="0.05"/>
-            </geometry>
-       <!--     <surface>
-              <friction>
-                <ode>
-                  <mu>0</mu>
-                  <mu2>0</mu2>
-                  <slip1>1.0</slip1>
-                  <slip2>1.0</slip2>
-                </ode>
-              </friction>
-            </surface> -->
-          </collision>
+  </link>
+    <joint name="caster_front_joint" type="fixed">
+      <parent link="base_link"/>
+      <child link="caster_front_link"/>
+      <origin xyz="0.2 0.0 -0.0385" rpy="${-M_PI/2} 0 0"/>
+    </joint>
+    <link name="caster_front_link">
+      <collision>
+        <geometry>
+          <cylinder length="0.0176" radius="0.05"/>
+        </geometry>
+        <origin rpy="0 0 0" xyz="0 0 0"/>
+      </collision>
+      <inertial>
+        <mass value="0.01" />
+        <origin xyz="0 0 0" />
+        <inertia ixx="0.001" ixy="0.0" ixz="0.0"
+                 iyy="0.001" iyz="0.0"
+                 izz="0.001" />
+      </inertial>
+    </link>
+    <joint name="caster_back_joint" type="fixed">
+      <parent link="base_link"/>
+      <child link="caster_back_link"/>
+      <origin xyz="-0.2 0.0 -0.0385" rpy="${-M_PI/2} 0 0"/>
+    </joint>
+    <link name="caster_back_link">
+      <collision>
+        <geometry>
+          <cylinder length="0.0176" radius="0.05"/>
+        </geometry>
+        <origin rpy="0 0 0" xyz="0 0 0"/>
+      </collision>
+      <inertial>
+        <mass value="0.01" />
+        <origin xyz="0 0 0" />
+        <inertia ixx="0.001" ixy="0.0" ixz="0.0"
+                 iyy="0.001" iyz="0.0"
+                 izz="0.001" />
+      </inertial>
+    </link>
+ <link
+    name="left_wheel_link">
+    <inertial>
+      <origin
+        xyz="9.16610941069373E-06 4.59070539915452E-09 8.0609835912647E-06"
+        rpy="0 0 0" />
+    <mass
+        value="1.8524" />
+      <inertia
+        ixx="0.0069046"
+        ixy="-3.8717E-08"
+        ixz="2.0707E-07"
+        iyy="0.013153"
+        iyz="-1.0124E-07"
+        izz="0.0069054" />
+      </inertial>
+    <visual>
+      <origin
+        xyz="0 0 0"
+        rpy="0 0 0" />
+      <geometry>
+        <mesh
+          filename="package://armadillo2_description/mesh/left_wheel_link.STL" />
+      </geometry>
+      <material
+        name="">
+        <color
+          rgba="0.792156862745098 0.819607843137255 0.933333333333333 1" />
+      </material>
+    </visual>
+    <collision>
+      <origin
+        xyz="0 0 0"
+        rpy="${M_PI/2} 0 0" />
+      <geometry>
+      <cylinder  length="0.04" radius="0.1"/>
+      </geometry>
+    </collision>
+  </link>
+  <joint
+    name="left_wheel_joint"
+    type="continuous">
+    <origin
+      xyz="0.063115 0.16085 0.0115"
+      rpy="0 0 0" />
+    <parent
+      link="base_link" />
+    <child
+      link="left_wheel_link" />
+    <axis
+      xyz="0 1 0" />
+    <limit
+      effort="0.1"
+      velocity="10.0" />
+  </joint>
+ <link
+    name="right_wheel_link">
+    <inertial>
+      <origin
+        xyz="9.16610941069373E-06 -4.99540929455033E-06 8.06098359126817E-06"
+        rpy="0 0 0" />
+       <mass
+        value="1.8524" />
+      <inertia
+        ixx="0.0069046"
+        ixy="-3.8717E-08"
+        ixz="-2.0707E-07"
+        iyy="0.013153"
+        iyz="1.0124E-07"
+        izz="0.0069054" />
+    </inertial>
+    <visual>
+      <origin
+        xyz="0 0 0"
+        rpy="0 0 0" />
+      <geometry>
+        <mesh
+          filename="package://armadillo2_description/mesh/right_wheel_link.STL" />
+      </geometry>
+      <material
+        name="">
+        <color
+          rgba="0.792156862745098 0.819607843137255 0.933333333333333 1" />
+      </material>
+    </visual>
+   <collision>
+      <origin
+        xyz="0 0 0"
+        rpy="${M_PI/2} 0 0" />
+      <geometry>
+      <cylinder  length="0.04" radius="0.1"/>
+      </geometry>
+    </collision>
+  </link>
+  <joint
+    name="right_wheel_joint"
+    type="continuous">
+    <origin
+      xyz="0.063115 -0.16085 0.0115"
+      rpy="0 0 0" />
+    <parent
+      link="base_link" />
+    <child
+      link="right_wheel_link" />
+    <axis
+      xyz="0 1 0" />
+    <limit
+      effort="0.1"
+      velocity="10.0" />
+  </joint>
+ <link
+    name="caster_left_link">
+    <visual>
+      <origin
+        xyz="0 0 0"
+        rpy="0 0 0" />
+      <geometry>
+        <mesh
+          filename="package://armadillo2_description/mesh/caster_left_link.STL" />
+      </geometry>
+      <material
+        name="">
+        <color
+          rgba="0.792156862745098 0.819607843137255 0.933333333333333 1" />
+      </material>
+    </visual>
   </link>
   <link
@@ -97,139 +245,4 @@
       xyz="0 0 0" />
   </joint>
- <link
-    name="left_wheel_link">
-    <inertial>
-      <origin
-        xyz="9.16610941069373E-06 4.59070539915452E-09 8.0609835912647E-06"
-        rpy="0 0 0" />
-      <mass
-        value="1.19468304707429" />
-      <inertia
-        ixx="0.00339394020641508"
-        ixy="-1.7040091442662E-11"
-        ixz="-3.19286008554441E-07"
-        iyy="0.00640943262315833"
-        iyz="-1.56330189682853E-11"
-        izz="0.00339385794108548" />
-    </inertial>
-    <visual>
-      <origin
-        xyz="0 0 0"
-        rpy="0 0 0" />
-      <geometry>
-        <mesh
-          filename="package://armadillo2_description/mesh/left_wheel_link.STL" />
-      </geometry>
-      <material
-        name="">
-        <color
-          rgba="0.792156862745098 0.819607843137255 0.933333333333333 1" />
-      </material>
-    </visual>
-    <collision>
-      <origin
-        xyz="0 0 0"
-        rpy="${M_PI/2} 0 0" />
-      <geometry>
-      <cylinder  length="0.04" radius="0.1"/>
-      </geometry>
-    </collision>
-  </link>
-  <joint
-    name="left_wheel_joint"
-    type="continuous">
-    <origin
-      xyz="0.063115 0.16085 0.0115"
-      rpy="0 0 0" />
-    <parent
-      link="base_link" />
-    <child
-      link="left_wheel_link" />
-    <axis
-      xyz="0 1 0" />
-  </joint>
- <link
-    name="right_wheel_link">
-    <inertial>
-      <origin
-        xyz="9.16610941069373E-06 -4.99540929455033E-06 8.06098359126817E-06"
-        rpy="0 0 0" />
-      <mass
-        value="1.19468304707429" />
-      <inertia
-        ixx="0.00339394020641508"
-        ixy="-1.70400914487861E-11"
-        ixz="-3.19286008554438E-07"
-        iyy="0.00640943262315833"
-        iyz="-1.5633018951093E-11"
-        izz="0.00339385794108548" />
-    </inertial>
-    <visual>
-      <origin
-        xyz="0 0 0"
-        rpy="0 0 0" />
-      <geometry>
-        <mesh
-          filename="package://armadillo2_description/mesh/right_wheel_link.STL" />
-      </geometry>
-      <material
-        name="">
-        <color
-          rgba="0.792156862745098 0.819607843137255 0.933333333333333 1" />
-      </material>
-    </visual>
-   <collision>
-      <origin
-        xyz="0 0 0"
-        rpy="${M_PI/2} 0 0" />
-      <geometry>
-      <cylinder  length="0.04" radius="0.1"/>
-      </geometry>
-    </collision>
-  </link>
-  <joint
-    name="right_wheel_joint"
-    type="continuous">
-    <origin
-      xyz="0.063115 -0.16085 0.0115"
-      rpy="0 0 0" />
-    <parent
-      link="base_link" />
-    <child
-      link="right_wheel_link" />
-    <axis
-      xyz="0 1 0" />
-  </joint>
- <link
-    name="caster_left_link">
-    <inertial>
-      <origin
-        xyz="0.00421271931699432 -3.85330403696038E-08 0.0101595051394297"
-        rpy="0 0 0" />
-      <mass
-        value="0.0496415739447828" />
-      <inertia
-        ixx="2.21176053576914E-05"
-        ixy="-1.28190365189921E-11"
-        ixz="5.51496344859667E-06"
-        iyy="2.871220501461E-05"
-        iyz="-3.35442196159029E-11"
-        izz="1.10273416039652E-05" />
-    </inertial>
-    <visual>
-      <origin
-        xyz="0 0 0"
-        rpy="0 0 0" />
-      <geometry>
-        <mesh
-          filename="package://armadillo2_description/mesh/caster_left_link.STL" />
-      </geometry>
-      <material
-        name="">
-        <color
-          rgba="0.792156862745098 0.819607843137255 0.933333333333333 1" />
-      </material>
-    </visual>
-  </link>
   <joint
     name="caster_left_joint"
@@ -247,18 +260,4 @@
   <link
     name="caster_right_link">
-    <inertial>
-      <origin
-        xyz="0.00421271931699441 -3.85330403973594E-08 0.0101595051394299"
-        rpy="0 0 0" />
-      <mass
-        value="0.049641573944783" />
-      <inertia
-        ixx="2.21176053576918E-05"
-        ixy="-1.28190365160225E-11"
-        ixz="5.5149634485968E-06"
-        iyy="2.87122050146104E-05"
-        iyz="-3.35442196090477E-11"
-        izz="1.10273416039652E-05" />
-    </inertial>
     <visual>
       <origin
@@ -291,17 +290,17 @@
   <link
     name="torso_link">
-    <inertial>
+  <inertial>
       <origin
         xyz="-0.059733 -0.00037419 0.54938"
         rpy="0 0 0" />
-      <mass
-        value="4.9226" />
-      <inertia
-        ixx="0.27696"
-        ixy="0.00010279"
-        ixz="-0.051125"
-        iyy="0.28305"
-        iyz="-5.4525E-06"
-        izz="0.10934" />
+     <mass
+        value="0.035511" />
+      <inertia
+        ixx="0.19579"
+        ixy="2.4285E-05"
+        ixz="-0.0045097"
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
File: armadillo2_description/urdf/armadillo2_gazebo.xacro (robot description, xacro)
@@ -1,5 +1,52 @@
 <?xml version="1.0"?>
-<robot xmlns:xacro="http://www.ros.org/wiki/xacro" name="armadillo_robot" description="ARMadillo Robot">
+<robot xmlns:xacro="http://www.ros.org/wiki/xacro" name="armadillo2_robot" description="ARMadillo2 Robot">
  <xacro:include filename="$(find armadillo2_description)/urdf/armadillo2.xacro" />
+<xacro:include filename="$(find armadillo2_gazebo)/macros/softkinetic_camera_ds325.xacro" />
+  <xacro:property name="URF_FOV" value="${10.0*M_PI/180}" />
+  <xacro:arg name="kinect2" default="true"/>
+  <xacro:arg name="kinect2_hz" default="30.0"/>
+  <xacro:arg name="kinect2_hd" default="false"/>
+  <xacro:arg name="kinect2_qhd" default="true"/>
+  <xacro:arg name="kinect2_sd" default="false"/>
+  <xacro:arg name="urf" default="true"/>
+  <xacro:arg name="imu" default="true"/>
+  <xacro:arg name="gps" default="true"/>
+  <xacro:arg name="lidar" default="true"/>
+  <xacro:arg name="softkinetic" default="true"/>
+   <!-- softkinetic -->
+  <xacro:if value="$(arg softkinetic)">
+     <xacro:softkinetic_gazebo name="softkinetic_rgb" ros_topic="softkinetic_camera"/>
+  </xacro:if>
+  <!-- kinect 2 -->
+  <xacro:if value="$(arg kinect2)">
+    <xacro:property name="kinect2_hz" value="$(arg kinect2_hz)"/>
+    <xacro:property name="kinect2_hd" value="$(arg kinect2_hd)"/>
+    <xacro:property name="kinect2_qhd" value="$(arg kinect2_qhd)"/>
+    <xacro:property name="kinect2_sd" value="$(arg kinect2_sd)"/>
+    <xacro:include filename="$(find armadillo2_gazebo)/macros/kinect2.xacro" />
+  </xacro:if>
+  <!-- Sonars -->
+  <xacro:if value="$(arg urf)">
+    <xacro:include filename="$(find armadillo2_gazebo)/macros/urf.xacro" />
+    <xacro:urf name="rear" link="front_urf_link" topic="URF/front" />
+  </xacro:if>
+  <!-- hokuyo   -->
+  <xacro:if value="$(arg lidar)">
+    <xacro:include filename="$(find armadillo2_gazebo)/macros/hokuyo.xacro" />
+    <xacro:lidar link="laser_link" topic="scan" samples="667" resolution="1" min_angle="-1.5707963" max_angle="1.5707963" range_min="0.05" range_max="10" range_resolution="0.01" />
+  </xacro:if>
+  <!-- GPS   -->
+  <xacro:if value="$(arg gps)">
+    <xacro:include filename="$(find armadillo2_gazebo)/macros/gps.xacro" />
+    <xacro:gps />
+  </xacro:if>
+  <!-- IMU   -->
+  <xacro:if value="$(arg imu)">
+    <xacro:include filename="$(find armadillo2_gazebo)/macros/imu.xacro" />
+    <xacro:imu link="base_link" imu_offset_x="0" imu_offset_y="0" imu_offset_z="${M_PI}"
+      imu_offset_roll="0" imu_offset_pitch="0"
+      imu_offset_yaw="0" mag_offset_x="0"
+      mag_offset_y="0" mag_offset_z="0" />
+    </xacro:if>
 <gazebo>
             <plugin name="gazebo_ros_control" filename="libgazebo_ros_control.so">
@@ -7,4 +54,47 @@
             </plugin>
           </gazebo>
+  <gazebo>
+     <plugin name="gazebo_grasp_fix" filename="libgazebo_grasp_fix.so">
+          <arm>
+             <arm_name>arm</arm_name>
+             <palm_link> wrist_link  </palm_link>
+             <gripper_link> left_finger_link </gripper_link>
+             <gripper_link> right_finger_link </gripper_link>
+          </arm>
+         <forces_angle_tolerance>100</forces_angle_tolerance>
+         <update_rate>50</update_rate>
+         <grip_count_threshold>4</grip_count_threshold>
+         <max_grip_count>8</max_grip_count>
+         <release_tolerance>0.005</release_tolerance>
+         <disable_collisions_on_attach>false</disable_collisions_on_attach>
+         <contact_topic>__default_topic__</contact_topic>
+      </plugin>
+  </gazebo>
+  <gazebo reference="left_finger_link">
+    <kp>1000000.0</kp>
+    <kd>100.0</kd>
+    <mu1>1.0</mu1>
+    <mu2>1.0</mu2>
+    <fdir1>0 0 1</fdir1>
+    <maxVel>1.0</maxVel>
+    <minDepth>0.00</minDepth>
+  </gazebo>
+  <gazebo reference="left_finger_joint">
+    <implicitSpringDamper>1</implicitSpringDamper>
+    <provideFeedback>1</provideFeedback>
+  </gazebo>
+  <gazebo reference="right_finger_link">
+    <kp>1000000.0</kp>
+    <kd>100.0</kd>
+    <mu1>1.0</mu1>
+    <mu2>1.0</mu2>
+    <fdir1>0 0 1</fdir1>
+    <maxVel>1.0</maxVel>
+    <minDepth>0.00</minDepth>
+  </gazebo>
+  <gazebo reference="right_finger_joint">
+    <implicitSpringDamper>1</implicitSpringDamper>
+    <provideFeedback>1</provideFeedback>
+  </gazebo>
           <transmission name="left_wheel_joint_trans">
             <type>transmission_interface/SimpleTransmission</type>
@@ -52,27 +142,40 @@
             </actuator>
           </transmission>
-          <gazebo reference="torso_joint_link">
-            <turnGravityOff>true</turnGravityOff>
-          </gazebo>
-<!--
-        <gazebo reference="left_wheel_link">
-          <kp>1000000.0</kp>
-          <kd>100.0</kd>
-          <mu1>1.5</mu1>
-          <mu2>1.5</mu2>
-          <fdir1>1 0 0</fdir1>
-          <maxVel>1.0</maxVel>
-          <minDepth>0.00</minDepth>
+      <gazebo reference="left_wheel_link">
+        <mu1>1.0</mu1>
+	    <mu2>1.0</mu2>
+	    <kp>1000000.0</kp>
+	    <kd>100.0</kd>
+	    <minDepth>0.001</minDepth>
+	    <maxVel>1.0</maxVel>
         </gazebo>
         <gazebo reference="right_wheel_link">
-          <kp>1000000.0</kp>
-          <kd>100.0</kd>
-          <mu1>1.5</mu1>
-          <mu2>1.5</mu2>
-          <fdir1>1 0 0</fdir1>
-          <maxVel>1.0</maxVel>
-          <minDepth>0.00</minDepth>
+        <mu1>1.0</mu1>
+	    <mu2>1.0</mu2>
+	    <kp>1000000.0</kp>
+	    <kd>100.0</kd>
+	    <minDepth>0.001</minDepth>
+	    <maxVel>1.0</maxVel>
         </gazebo>
-          -->
+	  <gazebo reference="caster_front_link">
+	    <mu1>0.0</mu1>
+	    <mu2>0.0</mu2>
+	    <kp>1000000.0</kp>
+	    <kd>100.0</kd>
+	    <minDepth>0.001</minDepth>
+	    <maxVel>1.0</maxVel>
+	  </gazebo>
+	  <gazebo reference="caster_back_link">
+	    <mu1>0.0</mu1>
+	    <mu2>0.0</mu2>
+	    <kp>1000000.0</kp>
+	    <kd>100.0</kd>
+	    <minDepth>0.001</minDepth>
+	    <maxVel>1.0</maxVel>
+	  </gazebo>
+	  <gazebo reference="base_link">
+	    <mu1>0.3</mu1>
+	    <mu2>0.3</mu2>
+	  </gazebo>
   <transmission name="rotation1_joint_trans">
     <type>transmission_interface/SimpleTransmission</type>

Commit message: pnp

File: armadillo2_description/urdf/armadillo2.xacro (robot description, xacro)
@@ -354,5 +354,5 @@
         rpy="0 0 0" />
       <mass
-        value="0.03653" />
+        value="0.003653" />
       <inertia
         ixx="3.6365E-05"
@@ -402,6 +402,6 @@
       upper="${3.1415926535897/3.0}"
       lower="${-3.1415926535897/3.0}"
-      effort="0.01"
-      velocity="2.016223585" />
+      effort="0.5"
+      velocity="2" />
 <dynamics damping="0.1" friction="0"/>
   </joint>
@@ -413,12 +413,12 @@
         rpy="0 0 0" />
       <mass
-        value="0.0232" />
-      <inertia
-        ixx="0.0056403"
+        value="0.00232" />
+      <inertia
+        ixx="0.00056403"
         ixy="-2.0419E-05"
         ixz="1.476E-05"
-        iyy="0.0012267"
+        iyy="0.00012267"
         iyz="1.5926E-07"
-        izz="0.0057848" />
+        izz="0.00057848" />
     </inertial>
     <visual>
@@ -461,6 +461,6 @@
     upper="${M_PI/3}"
     lower="${-M_PI/6}"
-      effort="0.01"
-      velocity="7.016223585" />
+      effort="0.5"
+      velocity="2" />
 <dynamics damping="0.1" friction="0"/>
   </joint>

File: armadillo2_description/urdf/armadillo2_gazebo.xacro (robot description, xacro)
@@ -67,5 +67,5 @@
          <max_grip_count>8</max_grip_count>
          <release_tolerance>0.005</release_tolerance>
-         <disable_collisions_on_attach>false</disable_collisions_on_attach>
+         <disable_collisions_on_attach>true</disable_collisions_on_attach>
          <contact_topic>__default_topic__</contact_topic>
       </plugin>

Commit message: adding moveit safety layer to torso

File: armadillo2_description/urdf/armadillo2.xacro (robot description, xacro)
@@ -318,5 +318,5 @@
       </material>
     </visual>
-    <collision>
+    <collision name="torso">
       <origin
         xyz="0 0 0"
@@ -325,4 +325,12 @@
         <mesh
           filename="package://armadillo2_description/mesh/torso_link.STL" />
+      </geometry>
+    </collision>
+     <collision name="safty box">
+      <origin
+        xyz="0 -0.03 0.9"
+        rpy="0 0 0" />
+      <geometry>
+<box size="0.07 0.5 0.8"/>
       </geometry>
     </collision>

Commit message: fixes

File: armadillo2_description/urdf/armadillo2.xacro (robot description, xacro)
@@ -929,9 +929,9 @@
       xyz="1 0 0" />
     <limit
-      effort="0.01"
+      effort="0.5"
       lower="-1.57"
       upper="1.57"
       velocity="0.1" />
-<dynamics damping="0.1" friction="0"/>
+<dynamics damping="0.5" friction="0.0"/>
   </joint>
   <link
@@ -988,9 +988,9 @@
       xyz="1 0 0" />
   <limit
-      effort="0.01"
+      effort="0.5"
       lower="-1.57"
       upper="1.57"
       velocity="0.1" />
-<dynamics damping="0.1" friction="0"/>
+<dynamics damping="0.5" friction="0.0"/>
   </joint>
   <link

File: armadillo2_description/urdf/armadillo2_gazebo.xacro (robot description, xacro)
@@ -64,5 +64,5 @@
          <max_grip_count>8</max_grip_count>
          <release_tolerance>0.005</release_tolerance>
-         <disable_collisions_on_attach>true</disable_collisions_on_attach>
+         <disable_collisions_on_attach>false</disable_collisions_on_attach>
          <contact_topic>__default_topic__</contact_topic>
       </plugin>

Commit message: pnp fix

File: armadillo2_description/urdf/armadillo2.xacro (robot description, xacro)
@@ -2,4 +2,5 @@
 <robot xmlns:xacro="http://www.ros.org/wiki/xacro" name="armadillo2_robot" description="ARMadillo2 Robot">
  <xacro:property name="M_PI" value="3.1415926535897931" />
+ <xacro:property name="WHEEL_RADIUS" value="0.095" />
  <xacro:include filename="$(find softkinetic_camera)/urdf/sofkinetic_ds325.xacro"/>
 <link name="base_footprint"/>
@@ -7,5 +8,5 @@
     <parent link="base_footprint"/>
     <child link="base_link"/>
-    <origin xyz="0.00 0.00 0.1" rpy="0.0 0.0 0.0"/>
+    <origin xyz="0.00 0.00 ${WHEEL_RADIUS-0.0115}" rpy="0.0 0.0 0.0"/>
   </joint>
   <link
@@ -51,5 +52,5 @@
       <parent link="base_link"/>
       <child link="caster_front_link"/>
-      <origin xyz="0.2 0.0 -0.0385" rpy="${-M_PI/2} 0 0"/>
+      <origin xyz="0.2 0.0 ${-WHEEL_RADIUS+0.0115+0.05}" rpy="${-M_PI/2} 0 0"/>
     </joint>
     <link name="caster_front_link">
@@ -71,5 +72,5 @@
       <parent link="base_link"/>
       <child link="caster_back_link"/>
-      <origin xyz="-0.2 0.0 -0.0385" rpy="${-M_PI/2} 0 0"/>
+      <origin xyz="-0.2 0.0 ${-WHEEL_RADIUS+0.0115+0.05}" rpy="${-M_PI/2} 0 0"/>
     </joint>
     <link name="caster_back_link">
@@ -123,5 +124,5 @@
         rpy="${M_PI/2} 0 0" />
       <geometry>
-      <cylinder  length="0.04" radius="0.1"/>
+      <cylinder  length="0.04" radius="${WHEEL_RADIUS}"/>
       </geometry>
     </collision>
@@ -178,5 +179,5 @@
         rpy="${M_PI/2} 0 0" />
       <geometry>
-      <cylinder  length="0.04" radius="0.1"/>
+      <cylinder  length="0.04" radius="${WHEEL_RADIUS}"/>
       </geometry>
     </collision>
@@ -868,5 +869,5 @@
       upper="3.14"
       velocity="2.0" />
-<dynamics damping="0.1" friction="0"/>
+<dynamics damping="0.5" friction="0.5"/>
   </joint>
   <link name="gripper_link"/>
@@ -933,5 +934,5 @@
       upper="1.57"
       velocity="0.1" />
-<dynamics damping="0.5" friction="0.0"/>
+<dynamics damping="0.5" friction="0.5"/>
   </joint>
   <link
@@ -992,5 +993,5 @@
       upper="1.57"
       velocity="0.1" />
-<dynamics damping="0.5" friction="0.0"/>
+<dynamics damping="0.5" friction="0.5"/>
   </joint>
   <link

File: armadillo2_description/urdf/armadillo2_gazebo.xacro (robot description, xacro)
@@ -70,10 +70,10 @@
   <gazebo reference="left_finger_link">
     <kp>1000000.0</kp>
-    <kd>100.0</kd>
+    <kd>1.0</kd>
     <mu1>1.0</mu1>
     <mu2>1.0</mu2>
     <fdir1>0 0 1</fdir1>
     <maxVel>1.0</maxVel>
-    <minDepth>0.00</minDepth>
+    <minDepth>0.001</minDepth>
   </gazebo>
   <gazebo reference="left_finger_joint">
@@ -83,10 +83,10 @@
   <gazebo reference="right_finger_link">
     <kp>1000000.0</kp>
-    <kd>100.0</kd>
+    <kd>1.0</kd>
     <mu1>1.0</mu1>
     <mu2>1.0</mu2>
     <fdir1>0 0 1</fdir1>
     <maxVel>1.0</maxVel>
-    <minDepth>0.00</minDepth>
+    <minDepth>0.001</minDepth>
   </gazebo>
   <gazebo reference="right_finger_joint">
