Commit message: calibrations of dxl vels

File: armadillo2_description/urdf/armadillo2.xacro (robot description, xacro)
@@ -409,6 +409,6 @@
       xyz="0 0 1" />
     <limit
-      upper="${3.1415926535897/3.0}"
-      lower="${-3.1415926535897/3.0}"
+      upper="${3.1415926535897/4.0}"
+      lower="${-3.1415926535897/4.0}"
       effort="0.5"
       velocity="2" />
@@ -468,5 +468,5 @@
       xyz="0 1 0" />
     <limit
-    upper="${M_PI/3}"
+    upper="${50.0*M_PI/180.0}"
     lower="${-M_PI/6}"
       effort="0.5"

File: armadillo2_description/urdf/armadillo2_gazebo.xacro (robot description, xacro)
@@ -16,5 +16,5 @@
    <!-- softkinetic -->
   <xacro:if value="$(arg softkinetic)">
-     <xacro:softkinetic_gazebo name="softkinetic_rgb" ros_topic="softkinetic_camera"/>
+     <xacro:softkinetic_gazebo name="softkinetic_rgb" ros_topic="softkinetic"/>
   </xacro:if>
   <!-- kinect 2 -->

File: armadillo2_utils/softkinetic/softkinetic_camera/urdf/sofkinetic_ds325.xacro (robot description, xacro)
@@ -5,5 +5,5 @@
     <!-- Add frames for RGB and depth optical axes -->
     <joint name="${name}_rgb_joint" type="fixed">
-      <origin xyz="0.02 -0.0125 0.0" rpy="0.0 0.0 0.0"/>
+      <origin xyz="0.025 -0.0125 0.0" rpy="0.0 0.0 0.0"/>
       <parent link="${name}_link"/>
       <child link="${name}_rgb_frame"/>

Commit message: adding stability to base while driving in gazebo

File: armadillo2_description/urdf/armadillo2.xacro (robot description, xacro)
@@ -49,10 +49,10 @@
           </collision>
   </link>
-    <joint name="caster_front_joint" type="fixed">
+    <joint name="caster_front_left_joint" type="fixed">
       <parent link="base_link"/>
-      <child link="caster_front_link"/>
-      <origin xyz="0.2 0.0 ${-WHEEL_RADIUS+0.0115+0.05}" rpy="${-M_PI/2} 0 0"/>
+      <child link="caster_front_left_link"/>
+      <origin xyz="0.2 0.24 ${-WHEEL_RADIUS+0.0115+0.05+0.005}" rpy="${-M_PI/2} 0 0"/>
     </joint>
-    <link name="caster_front_link">
+    <link name="caster_front_left_link">
       <collision>
         <geometry>
@@ -69,10 +69,50 @@
       </inertial>
     </link>
-    <joint name="caster_back_joint" type="fixed">
+    <joint name="caster_back_left_joint" type="fixed">
       <parent link="base_link"/>
-      <child link="caster_back_link"/>
-      <origin xyz="-0.2 0.0 ${-WHEEL_RADIUS+0.0115+0.05}" rpy="${-M_PI/2} 0 0"/>
+      <child link="caster_back_left_link"/>
+      <origin xyz="-0.2 0.24 ${-WHEEL_RADIUS+0.0115+0.05}" rpy="${-M_PI/2} 0 0"/>
     </joint>
-    <link name="caster_back_link">
+    <link name="caster_back_left_link">
+      <collision>
+        <geometry>
+          <cylinder length="0.0176" radius="0.05"/>
+        </geometry>
+        <origin rpy="0 0 0" xyz="0 0 0"/>
+      </collision>
+      <inertial>
+        <mass value="0.01" />
+        <origin xyz="0 0 0" />
+        <inertia ixx="0.001" ixy="0.0" ixz="0.0"
+                 iyy="0.001" iyz="0.0"
+                 izz="0.001" />
+      </inertial>
+    </link>
+        <joint name="caster_front_right_joint" type="fixed">
+      <parent link="base_link"/>
+      <child link="caster_front_right_link"/>
+      <origin xyz="0.2 -0.24 ${-WHEEL_RADIUS+0.0115+0.05+0.005}" rpy="${-M_PI/2} 0 0"/>
+    </joint>
+    <link name="caster_front_right_link">
+      <collision>
+        <geometry>
+          <cylinder length="0.0176" radius="0.05"/>
+        </geometry>
+        <origin rpy="0 0 0" xyz="0 0 0"/>
+      </collision>
+      <inertial>
+        <mass value="0.01" />
+        <origin xyz="0 0 0" />
+        <inertia ixx="0.001" ixy="0.0" ixz="0.0"
+                 iyy="0.001" iyz="0.0"
+                 izz="0.001" />
+      </inertial>
+    </link>
+    <joint name="caster_back_right_joint" type="fixed">
+      <parent link="base_link"/>
+      <child link="caster_back_right_link"/>
+      <origin xyz="-0.2 -0.24 ${-WHEEL_RADIUS+0.0115+0.05}" rpy="${-M_PI/2} 0 0"/>
+    </joint>
+    <link name="caster_back_right_link">
       <collision>
         <geometry>

File: armadillo2_description/urdf/armadillo2_gazebo.xacro (robot description, xacro)
@@ -154,13 +154,29 @@
         <maxVel>1.0</maxVel>
     </gazebo>
-    <gazebo reference="caster_front_link">
-        <mu1>0.0</mu1>
-        <mu2>0.0</mu2>
-        <kp>1000000.0</kp>
-        <kd>100.0</kd>
-        <minDepth>0.001</minDepth>
-        <maxVel>1.0</maxVel>
-    </gazebo>
-    <gazebo reference="caster_back_link">
+    <gazebo reference="caster_front_right_link">
+        <mu1>0.0</mu1>
+        <mu2>0.0</mu2>
+        <kp>1000000.0</kp>
+        <kd>100.0</kd>
+        <minDepth>0.001</minDepth>
+        <maxVel>1.0</maxVel>
+    </gazebo>
+    <gazebo reference="caster_back_right_link">
+        <mu1>0.0</mu1>
+        <mu2>0.0</mu2>
+        <kp>1000000.0</kp>
+        <kd>100.0</kd>
+        <minDepth>0.001</minDepth>
+        <maxVel>1.0</maxVel>
+    </gazebo>
+        <gazebo reference="caster_front_left_link">
+        <mu1>0.0</mu1>
+        <mu2>0.0</mu2>
+        <kp>1000000.0</kp>
+        <kd>100.0</kd>
+        <minDepth>0.001</minDepth>
+        <maxVel>1.0</maxVel>
+    </gazebo>
+    <gazebo reference="caster_back_left_link">
         <mu1>0.0</mu1>
         <mu2>0.0</mu2>

Commit message: lowering arm mass for more driving stability in az

File: armadillo2_description/urdf/armadillo2.xacro (robot description, xacro)
@@ -564,5 +564,5 @@
         rpy="0 0 0" />
       <mass
-        value="0.0035317" />
+        value="0.0000017" />
       <inertia
         ixx="0.00055596"
@@ -623,5 +623,5 @@
         rpy="0 0 0" />
       <mass
-        value="0.0052217" />
+        value="0.0000017" />
       <inertia
         ixx="0.0043595"
@@ -682,5 +682,5 @@
         rpy="0 0 0" />
       <mass
-        value="0.0047392" />
+        value="0.0000017" />
       <inertia
         ixx="0.00093237"
@@ -741,5 +741,5 @@
         rpy="0 0 0" />
       <mass
-        value="0.001635" />
+        value="0.0000017" />
       <inertia
         ixx="0.00014092"
@@ -800,5 +800,5 @@
         rpy="0 0 0" />
       <mass
-        value="0.0015954" />
+        value="0.0000017" />
       <inertia
         ixx="0.00018198"
@@ -859,5 +859,5 @@
         rpy="0 0 0" />
       <mass
-        value="0.0011365" />
+        value="0.0000017" />
       <inertia
         ixx="4.4099E-05"
@@ -924,5 +924,5 @@
         rpy="0 0 0" />
       <mass
-        value="0.0017229" />
+        value="0.0000017" />
       <inertia
         ixx="1.4683E-05"
@@ -983,5 +983,5 @@
         rpy="0 0 0" />
       <mass
-        value="0.0017229" />
+        value="0.0000017" />
       <inertia
         ixx="1.4683E-05"
@@ -1037,4 +1037,18 @@
   <link
     name="softkinetic_link">
+    <inertial>
+      <origin
+        xyz="-1.1102E-16 -0.015598 0.034754"
+        rpy="0 0 0" />
+      <mass
+        value="0.0000017" />
+      <inertia
+        ixx="1.4683E-05"
+        ixy="2.0869E-20"
+        ixz="-3.5787E-20"
+        iyy="1.7304E-05"
+        iyz="-9.2811E-07"
+        izz="4.5506E-06" />
+    </inertial>
     <visual>
       <origin

Commit message: arm tuning

File: armadillo2_description/urdf/armadillo2.xacro (robot description, xacro)
@@ -373,5 +373,5 @@
         rpy="0 0 0" />
       <geometry>
-<box size="0.07 0.5 0.8"/>
+        <box size="0.09 0.5 0.8"/>
       </geometry>
     </collision>

Commit message: Update armadillo2.xacro

File: armadillo2_description/urdf/armadillo2.xacro (robot description, xacro)
@@ -16,12 +16,12 @@
         xyz="-0.012353 0.000122 0.17716"
         rpy="0 0 0" />
-       <mass value="30.65"/>
+       <mass value="100.65"/>
        <inertia
-        ixx="0.61639"
+        ixx="0.31639"
         ixy="-9.1727E-05"
         ixz="-0.093044"
-        iyy="0.57997"
+        iyy="0.17997"
         iyz="5.3231E-05"
-        izz="0.36693" />
+        izz="0.16693" />
     </inertial>
     <visual>
@@ -52,5 +52,5 @@
       <parent link="base_link"/>
       <child link="caster_front_left_link"/>
-      <origin xyz="0.2 0.24 ${-WHEEL_RADIUS+0.0115+0.05+0.005}" rpy="${-M_PI/2} 0 0"/>
+      <origin xyz="0.2 0.24 ${-WHEEL_RADIUS+0.0115+0.05+0.015}" rpy="${-M_PI/2} 0 0"/>
     </joint>
     <link name="caster_front_left_link">
@@ -92,5 +92,5 @@
       <parent link="base_link"/>
       <child link="caster_front_right_link"/>
-      <origin xyz="0.2 -0.24 ${-WHEEL_RADIUS+0.0115+0.05+0.005}" rpy="${-M_PI/2} 0 0"/>
+      <origin xyz="0.2 -0.24 ${-WHEEL_RADIUS+0.0115+0.05+0.015}" rpy="${-M_PI/2} 0 0"/>
     </joint>
     <link name="caster_front_right_link">
@@ -338,8 +338,8 @@
         value="0.035511" />
       <inertia
-        ixx="0.19579"
+        ixx="0.09579"
         ixy="2.4285E-05"
         ixz="-0.0045097"
-        iyy="0.16807"
+        iyy="0.06807"
         iyz="-7.4938E-05"
         izz="0.072852" />
@@ -516,4 +516,18 @@
   <link
     name="kinect2_link" />
+   <inertial>
+      <origin
+        xyz="0.014321 0.00038338 0.064622"
+        rpy="0 0 0" />
+      <mass
+        value="0.00232" />
+      <inertia
+        ixx="0.00056403"
+        ixy="-2.0419E-05"
+        ixz="1.476E-05"
+        iyy="0.00012267"
+        iyz="1.5926E-07"
+        izz="0.00057848" />
+    </inertial>
   <joint
     name="kinect2_joint"

Commit message: added intel cam to gazebo --tested ok

File: armadillo2_description/urdf/armadillo2.xacro (robot description, xacro)
@@ -3,5 +3,4 @@
  <xacro:property name="M_PI" value="3.1415926535897931" />
  <xacro:property name="WHEEL_RADIUS" value="0.095" />
- <xacro:include filename="$(find softkinetic_camera)/urdf/sofkinetic_ds325.xacro"/>
 <link name="base_footprint"/>
  <joint name="base_footprint_joint" type="fixed">
@@ -1050,5 +1049,5 @@
   </joint>
   <link
-    name="softkinetic_link">
+    name="intel_d435_link">
     <inertial>
       <origin
@@ -1067,6 +1066,6 @@
     <visual>
       <origin
-        xyz="0 0 0"
-        rpy="0 0 0" />
+        xyz="-0.013021 0.04474 -0.012"
+        rpy="0 0 -1.5708" />
       <geometry>
         <mesh
@@ -1090,18 +1089,74 @@
   </link>
   <joint
-    name="softkinetic_joint"
+    name="intel_d435_joint"
     type="fixed">
     <origin
-      xyz="0.04474 0.0 -0.037"
-      rpy="-3.1416 0 3.1416" />
+      xyz="0 0.0143 -0.049"
+      rpy="-3.1416 0 1.5708" />
     <parent
       link="wrist_link" />
     <child
-      link="softkinetic_link" />
+      link="intel_d435_link" />
     <axis
       xyz="0 0 0" />
-  </joint>
-<softkinetic_camera name="softkinetic" >
-    <origin xyz="-0.05905 0 0.0753" rpy="0.0 -${M_PI/2} 0.0"/>
-</softkinetic_camera>
+    </joint>
+<!--
+License: Apache 2.0. See LICENSE file in root directory.
+Copyright(c) 2017 Intel Corporation. All Rights Reserved
+the following is the URDF model for the Intel RealSense 430 intel_d435, in it's
+aluminum peripherial evaluation case.
+Edited by RoboTiCan
+-->
+    <!-- camera depth joints and links -->
+    <joint name="intel_d435_depth_joint" type="fixed">
+      <origin xyz="0 -0.0122 0" rpy="0 0 0"/>
+      <parent link="intel_d435_link"/>
+      <child link="intel_d435_depth_frame" />
+    </joint>
+    <link name="intel_d435_depth_frame"/>
+    <joint name="intel_d435_depth_optical_joint" type="fixed">
+      <origin xyz="0.0125 0 0.0" rpy="${-M_PI/2} 0 ${-M_PI/2}" />
+      <parent link="intel_d435_depth_frame" />
+      <child link="intel_d435_depth_optical_frame" />
+    </joint>
+    <link name="intel_d435_depth_optical_frame"/>
+    <!-- intel_d435 left IR joints and links -->
+    <joint name="intel_d435_left_ir_joint" type="fixed">
+      <origin xyz="0 -0.0322 0" rpy="0 0 0" />
+      <parent link="intel_d435_link" />
+      <child link="intel_d435_left_ir_frame" />
+    </joint>
+    <link name="intel_d435_left_ir_frame"/>
+    <joint name="intel_d435_left_ir_optical_joint" type="fixed">
+      <origin xyz="0.0125 0 0" rpy="${-M_PI/2} 0 ${-M_PI/2}" />
+      <parent link="intel_d435_left_ir_frame" />
+      <child link="intel_d435_left_ir_optical_frame" />
+    </joint>
+    <link name="intel_d435_left_ir_optical_frame"/>
+    <!-- intel_d435 right IR joints and links -->
+    <joint name="intel_d435_right_ir_joint" type="fixed">
+      <origin xyz="0 0.0178 0" rpy="0 0 0" />
+      <parent link="intel_d435_link" />
+      <child link="intel_d435_right_ir_frame" />
+    </joint>
+    <link name="intel_d435_right_ir_frame"/>
+    <joint name="intel_d435_right_ir_optical_joint" type="fixed">
+      <origin xyz="0.0125 0 0" rpy="${-M_PI/2} 0 ${-M_PI/2}" />
+      <parent link="intel_d435_right_ir_frame" />
+      <child link="intel_d435_right_ir_optical_frame" />
+    </joint>
+    <link name="intel_d435_right_ir_optical_frame"/>
+    <!-- intel_d435 fisheye joints and links -->
+    <joint name="intel_d435_fisheye_joint" type="fixed">
+      <origin xyz="0 0.0322 0" rpy="0 0 0" />
+      <parent link="intel_d435_link" />
+      <child link="intel_d435_fisheye_frame" />
+    </joint>
+    <link name="intel_d435_fisheye_frame"/>
+    <joint name="intel_d435_fisheye_optical_joint" type="fixed">
+      <origin xyz="0.0125 0 0" rpy="${-M_PI/2} 0 ${-M_PI/2}" />
+      <parent link="intel_d435_fisheye_frame" />
+      <child link="intel_d435_fisheye_optical_frame" />
+    </joint>
+    <link name="intel_d435_fisheye_optical_frame"/>
 </robot>

File: armadillo2_description/urdf/armadillo2_gazebo.xacro (robot description, xacro)
@@ -2,5 +2,5 @@
 <robot xmlns:xacro="http://www.ros.org/wiki/xacro" name="armadillo2_robot" description="ARMadillo2 Robot">
     <xacro:include filename="$(find armadillo2_description)/urdf/armadillo2.xacro" />
-    <xacro:include filename="$(find armadillo2_gazebo)/macros/softkinetic_camera_ds325.xacro" />
+    <xacro:include filename="$(find armadillo2_gazebo)/macros/intel_cam.xacro" />
     <xacro:arg name="kinect2" default="true"/>
     <xacro:arg name="kinect2_hz" default="30.0"/>
@@ -12,8 +12,9 @@
     <xacro:arg name="gps" default="true"/>
     <xacro:arg name="lidar" default="true"/>
-    <xacro:arg name="softkinetic" default="true"/>
-    <!-- softkinetic -->
-    <xacro:if value="$(arg softkinetic)">
-        <xacro:softkinetic_gazebo name="softkinetic_rgb" ros_topic="softkinetic"/>
+    <xacro:arg name="intel_cam" default="true"/>
+    <!-- intel_cam -->
+    <xacro:if value="$(arg intel_cam)">
+        <xacro:include filename="$(find armadillo2_gazebo)/macros/intel_cam.xacro" />
+        <xacro:intel_d435_gazebo name="intel_d435" ros_topic="intel_cam"/>
     </xacro:if>
     <!-- kinect 2 -->

Commit message: replacing intel cam mesh, refactoring xacro

File: armadillo2_description/urdf/armadillo2.xacro (robot description, xacro)
@@ -3,4 +3,5 @@
  <xacro:property name="M_PI" value="3.1415926535897931" />
  <xacro:property name="WHEEL_RADIUS" value="0.095" />
+ <xacro:include filename="$(find armadillo2_description)/urdf/intel_d435.urdf"/>
 <link name="base_footprint"/>
  <joint name="base_footprint_joint" type="fixed">
@@ -1048,45 +1049,5 @@
 <dynamics damping="0.5" friction="0.5"/>
   </joint>
-  <link
-    name="intel_d435_link">
-    <inertial>
-      <origin
-        xyz="-1.1102E-16 -0.015598 0.034754"
-        rpy="0 0 0" />
-      <mass
-        value="0.0000017" />
-      <inertia
-        ixx="1.4683E-05"
-        ixy="2.0869E-20"
-        ixz="-3.5787E-20"
-        iyy="1.7304E-05"
-        iyz="-9.2811E-07"
-        izz="4.5506E-06" />
-    </inertial>
-    <visual>
-      <origin
-        xyz="-0.013021 0.04474 -0.012"
-        rpy="0 0 -1.5708" />
-      <geometry>
-        <mesh
-          filename="package://armadillo2_description/mesh/intel_d435.STL" />
-      </geometry>
-      <material
-        name="">
-        <color
-          rgba="0.25098 0.25098 0.25098 1" />
-      </material>
-    </visual>
-    <collision>
-      <origin
-        xyz="0 0 0"
-        rpy="0 0 0" />
-      <geometry>
-        <mesh
-          filename="package://armadillo2_description/mesh/intel_d435.STL" />
-      </geometry>
-    </collision>
-  </link>
-  <joint
+ <!-- <joint
     name="intel_d435_joint"
     type="fixed">
@@ -1100,63 +1061,57 @@
     <axis
       xyz="0 0 0" />
-    </joint>
-<!--
-License: Apache 2.0. See LICENSE file in root directory.
-Copyright(c) 2017 Intel Corporation. All Rights Reserved
-the following is the URDF model for the Intel RealSense 430 intel_d435, in it's
-aluminum peripherial evaluation case.
-Edited by RoboTiCan
--->
-    <!-- camera depth joints and links -->
-    <joint name="intel_d435_depth_joint" type="fixed">
-      <origin xyz="0 -0.0122 0" rpy="0 0 0"/>
-      <parent link="intel_d435_link"/>
-      <child link="intel_d435_depth_frame" />
-    </joint>
-    <link name="intel_d435_depth_frame"/>
-    <joint name="intel_d435_depth_optical_joint" type="fixed">
-      <origin xyz="0.0125 0 0.0" rpy="${-M_PI/2} 0 ${-M_PI/2}" />
-      <parent link="intel_d435_depth_frame" />
-      <child link="intel_d435_depth_optical_frame" />
-    </joint>
-    <link name="intel_d435_depth_optical_frame"/>
-    <!-- intel_d435 left IR joints and links -->
-    <joint name="intel_d435_left_ir_joint" type="fixed">
-      <origin xyz="0 -0.0322 0" rpy="0 0 0" />
-      <parent link="intel_d435_link" />
-      <child link="intel_d435_left_ir_frame" />
-    </joint>
-    <link name="intel_d435_left_ir_frame"/>
-    <joint name="intel_d435_left_ir_optical_joint" type="fixed">
-      <origin xyz="0.0125 0 0" rpy="${-M_PI/2} 0 ${-M_PI/2}" />
-      <parent link="intel_d435_left_ir_frame" />
-      <child link="intel_d435_left_ir_optical_frame" />
-    </joint>
-    <link name="intel_d435_left_ir_optical_frame"/>
-    <!-- intel_d435 right IR joints and links -->
-    <joint name="intel_d435_right_ir_joint" type="fixed">
-      <origin xyz="0 0.0178 0" rpy="0 0 0" />
-      <parent link="intel_d435_link" />
-      <child link="intel_d435_right_ir_frame" />
-    </joint>
-    <link name="intel_d435_right_ir_frame"/>
-    <joint name="intel_d435_right_ir_optical_joint" type="fixed">
-      <origin xyz="0.0125 0 0" rpy="${-M_PI/2} 0 ${-M_PI/2}" />
-      <parent link="intel_d435_right_ir_frame" />
-      <child link="intel_d435_right_ir_optical_frame" />
-    </joint>
-    <link name="intel_d435_right_ir_optical_frame"/>
-    <!-- intel_d435 fisheye joints and links -->
-    <joint name="intel_d435_fisheye_joint" type="fixed">
-      <origin xyz="0 0.0322 0" rpy="0 0 0" />
-      <parent link="intel_d435_link" />
-      <child link="intel_d435_fisheye_frame" />
-    </joint>
-    <link name="intel_d435_fisheye_frame"/>
-    <joint name="intel_d435_fisheye_optical_joint" type="fixed">
-      <origin xyz="0.0125 0 0" rpy="${-M_PI/2} 0 ${-M_PI/2}" />
-      <parent link="intel_d435_fisheye_frame" />
-      <child link="intel_d435_fisheye_optical_frame" />
-    </joint>
-    <link name="intel_d435_fisheye_optical_frame"/>
+    </joint>-->
+  <link
+    name="intel_d435_link">
+    <inertial>
+      <origin
+        xyz="0.00209672590490473 0.00107373429916791 -0.0124264025663287"
+        rpy="0 0 0" />
+      <mass
+        value="0.0446256012085417" />
+      <inertia
+        ixx="2.62358816469287E-05"
+        ixy="3.51148589025883E-07"
+        ixz="3.91275343984781E-11"
+        iyy="4.02618646244092E-06"
+        iyz="-6.05255657169474E-09"
+        izz="2.64982132448102E-05" />
+    </inertial>
+    <visual>
+      <origin
+        xyz="0 0 0.0125"
+        rpy="0 0 0" />
+      <geometry>
+        <mesh
+          filename="package://armadillo2_description/mesh/intel_d435.STL" />
+      </geometry>
+      <material
+        name="">
+        <color
+          rgba="0.792156862745098 0.819607843137255 0.933333333333333 1" />
+      </material>
+    </visual>
+    <collision>
+      <origin
+        xyz="0 0 0"
+        rpy="0 0 0" />
+      <geometry>
+        <mesh
+          filename="package://armadillo2_description/mesh/intel_d435.STL" />
+      </geometry>
+    </collision>
+  </link>
+    <joint
+    name="intel_d435_joint"
+    type="fixed">
+    <origin
+      xyz="0 0.0143 -0.0495"
+      rpy="-3.1416 6.1062E-16 1.5708" />
+    <parent
+      link="wrist_link" />
+    <child
+      link="intel_d435_link" />
+    <axis
+      xyz="0 0 0" />
+  </joint>
 </robot>
