Commit message: intel_d435 updates

File: armadillo2_description/urdf/armadillo2.xacro (robot description, xacro)
@@ -1062,5 +1062,5 @@
       xyz="0 0 0" />
     </joint>-->
-  <link
+  <!--<link
     name="intel_d435_link">
     <inertial>
@@ -1101,5 +1101,5 @@
       </geometry>
     </collision>
-  </link>
+  </link>-->
     <joint
     name="intel_d435_joint"
@@ -1111,5 +1111,5 @@
       link="wrist_link" />
     <child
-      link="intel_d435_link" />
+      link="camera_link" />
     <axis
       xyz="0 0 0" />

File: armadillo2_description/urdf/armadillo2_gazebo.xacro (robot description, xacro)
@@ -16,5 +16,5 @@
     <xacro:if value="$(arg intel_cam)">
         <xacro:include filename="$(find armadillo2_gazebo)/macros/intel_cam.xacro" />
-        <xacro:intel_d435_gazebo name="intel_d435" ros_topic="intel_cam"/>
+        <xacro:intel_d435_gazebo name="camera" ros_topic="intel_cam"/>
     </xacro:if>
     <!-- kinect 2 -->

File: armadillo2_description/urdf/intel_d435.urdf (robot description, URDF)
Before this commit: robot intel_d435, 8 links, 8 joints
Links:
- removed link intel_d435_depth_frame
- removed link intel_d435_depth_optical_frame
- removed link intel_d435_fisheye_frame
- removed link intel_d435_fisheye_optical_frame
- removed link intel_d435_left_ir_frame
- removed link intel_d435_left_ir_optical_frame
- removed link intel_d435_right_ir_frame
- removed link intel_d435_right_ir_optical_frame
- added link camera_depth_frame
- added link camera_depth_optical_frame
- added link camera_fisheye_frame
- added link camera_fisheye_optical_frame
- added link camera_left_ir_frame
- added link camera_left_ir_optical_frame
- added link camera_link, mass 0.0446256012085417; collision mesh filename=package://armadillo2_description/mesh/intel_d435.STL; visual mesh filename=package://armadillo2_description/mesh/intel_d435.STL
- added link camera_right_ir_frame
- added link camera_right_ir_optical_frame
Joints:
- removed joint intel_d435_depth_joint
- removed joint intel_d435_depth_optical_joint
- removed joint intel_d435_fisheye_joint
- removed joint intel_d435_fisheye_optical_joint
- removed joint intel_d435_left_ir_joint
- removed joint intel_d435_left_ir_optical_joint
- removed joint intel_d435_right_ir_joint
- removed joint intel_d435_right_ir_optical_joint
- added joint camera_depth_joint: type fixed, parent camera_link, child camera_depth_frame, origin xyz=0 -0.0122 0 rpy=0 0 0
- added joint camera_depth_optical_joint: type fixed, parent camera_depth_frame, child camera_depth_optical_frame, origin xyz=0 0 0 rpy=${-M_PI/2} 0 ${-M_PI/2}
- added joint camera_fisheye_joint: type fixed, parent camera_link, child camera_fisheye_frame, origin xyz=0 0.0322 0 rpy=0 0 0
- added joint camera_fisheye_optical_joint: type fixed, parent camera_fisheye_frame, child camera_fisheye_optical_frame, origin xyz=0 0 0 rpy=${-M_PI/2} 0 ${-M_PI/2}
- added joint camera_left_ir_joint: type fixed, parent camera_link, child camera_left_ir_frame, origin xyz=0 -0.0322 0 rpy=0 0 0
- added joint camera_left_ir_optical_joint: type fixed, parent camera_left_ir_frame, child camera_left_ir_optical_frame, origin xyz=0 0 0 rpy=${-M_PI/2} 0 ${-M_PI/2}
- added joint camera_right_ir_joint: type fixed, parent camera_link, child camera_right_ir_frame, origin xyz=0 0.0178 0 rpy=0 0 0
- added joint camera_right_ir_optical_joint: type fixed, parent camera_right_ir_frame, child camera_right_ir_optical_frame, origin xyz=0 0 0 rpy=${-M_PI/2} 0 ${-M_PI/2}

File: armadillo2_gazebo/macros/intel_cam.xacro (robot description, xacro)
@@ -24,5 +24,5 @@
              <alwaysOn>true</alwaysOn>
                 <updateRate>10.0</updateRate>
-                <cameraName>${name}</cameraName>
+                <cameraName>${ros_topic}</cameraName>
                 <frameName>${name}_depth_optical_frame</frameName>
             <imageTopicName>color/image_raw</imageTopicName>

Commit message: updating robot model masses for gazebo

File: armadillo2_description/urdf/armadillo2.xacro (robot description, xacro)
@@ -16,5 +16,5 @@
         xyz="-0.012353 0.000122 0.17716"
         rpy="0 0 0" />
-       <mass value="100.65"/>
+       <mass value="100.0"/>
        <inertia
         ixx="0.31639"
@@ -578,5 +578,5 @@
         rpy="0 0 0" />
       <mass
-        value="0.0000017" />
+        value="0.5" />
       <inertia
         ixx="0.00055596"
@@ -637,5 +637,5 @@
         rpy="0 0 0" />
       <mass
-        value="0.0000017" />
+        value="0.5" />
       <inertia
         ixx="0.0043595"
@@ -696,5 +696,5 @@
         rpy="0 0 0" />
       <mass
-        value="0.0000017" />
+        value="0.5" />
       <inertia
         ixx="0.00093237"
@@ -755,5 +755,5 @@
         rpy="0 0 0" />
       <mass
-        value="0.0000017" />
+        value="0.3" />
       <inertia
         ixx="0.00014092"
@@ -814,5 +814,5 @@
         rpy="0 0 0" />
       <mass
-        value="0.0000017" />
+        value="0.3" />
       <inertia
         ixx="0.00018198"
@@ -873,5 +873,5 @@
         rpy="0 0 0" />
       <mass
-        value="0.0000017" />
+        value="0.3" />
       <inertia
         ixx="4.4099E-05"
@@ -938,5 +938,5 @@
         rpy="0 0 0" />
       <mass
-        value="0.0000017" />
+        value="0.1" />
       <inertia
         ixx="1.4683E-05"
@@ -997,5 +997,5 @@
         rpy="0 0 0" />
       <mass
-        value="0.0000017" />
+        value="0.1" />
       <inertia
         ixx="1.4683E-05"

Commit message: adding armadillo2.0 files

File: armadillo2_description/urdf/armadillo2.xacro (robot description, xacro)
@@ -3,5 +3,5 @@
  <xacro:property name="M_PI" value="3.1415926535897931" />
  <xacro:property name="WHEEL_RADIUS" value="0.095" />
- <xacro:include filename="$(find armadillo2_description)/urdf/intel_d435.urdf"/>
+ <xacro:include filename="$(find softkinetic_camera)/urdf/sofkinetic_ds325.xacro"/>
 <link name="base_footprint"/>
  <joint name="base_footprint_joint" type="fixed">
@@ -1049,69 +1049,59 @@
 <dynamics damping="0.5" friction="0.5"/>
   </joint>
- <!-- <joint
-    name="intel_d435_joint"
+  <link
+    name="softkinetic_link">
+    <inertial>
+      <origin
+        xyz="-1.1102E-16 -0.015598 0.034754"
+        rpy="0 0 0" />
+      <mass
+        value="0.0000017" />
+      <inertia
+        ixx="1.4683E-05"
+        ixy="2.0869E-20"
+        ixz="-3.5787E-20"
+        iyy="1.7304E-05"
+        iyz="-9.2811E-07"
+        izz="4.5506E-06" />
+    </inertial>
+    <visual>
+      <origin
+        xyz="0 0 0"
+        rpy="0 0 0" />
+      <geometry>
+        <mesh
+          filename="package://armadillo2_description/mesh/softkinetic_link.STL" />
+      </geometry>
+      <material
+        name="">
+        <color
+          rgba="0.25098 0.25098 0.25098 1" />
+      </material>
+    </visual>
+    <collision>
+      <origin
+        xyz="0 0 0"
+        rpy="0 0 0" />
+      <geometry>
+        <mesh
+          filename="package://armadillo2_description/mesh/softkinetic_link.STL" />
+      </geometry>
+    </collision>
+  </link>
+  <joint
+    name="softkinetic_joint"
     type="fixed">
     <origin
-      xyz="0 0.0143 -0.049"
-      rpy="-3.1416 0 1.5708" />
+      xyz="0 0.0143 -0.0598"
+      rpy="-3.1416 6.1062E-16 1.5708" />
     <parent
       link="wrist_link" />
     <child
-      link="intel_d435_link" />
+      link="softkinetic_link" />
     <axis
       xyz="0 0 0" />
-    </joint>-->
-  <!--<link
-    name="intel_d435_link">
-    <inertial>
-      <origin
-        xyz="0.00209672590490473 0.00107373429916791 -0.0124264025663287"
-        rpy="0 0 0" />
-      <mass
-        value="0.0446256012085417" />
-      <inertia
-        ixx="2.62358816469287E-05"
-        ixy="3.51148589025883E-07"
-        ixz="3.91275343984781E-11"
-        iyy="4.02618646244092E-06"
-        iyz="-6.05255657169474E-09"
-        izz="2.64982132448102E-05" />
-    </inertial>
-    <visual>
-      <origin
-        xyz="0 0 0.0125"
-        rpy="0 0 0" />
-      <geometry>
-        <mesh
-          filename="package://armadillo2_description/mesh/intel_d435.STL" />
-      </geometry>
-      <material
-        name="">
-        <color
-          rgba="0.792156862745098 0.819607843137255 0.933333333333333 1" />
-      </material>
-    </visual>
-    <collision>
-      <origin
-        xyz="0 0 0"
-        rpy="0 0 0" />
-      <geometry>
-        <mesh
-          filename="package://armadillo2_description/mesh/intel_d435.STL" />
-      </geometry>
-    </collision>
-  </link>-->
-    <joint
-    name="intel_d435_joint"
-    type="fixed">
-    <origin
-      xyz="0 0.0143 -0.0495"
-      rpy="-3.1416 6.1062E-16 1.5708" />
-    <parent
-      link="wrist_link" />
-    <child
-      link="camera_link" />
-    <axis
-      xyz="0 0 0" />
-  </joint>
+  </joint>
+<softkinetic_camera name="softkinetic" >
+    <origin xyz="-0.05905 0 0.0753" rpy="0.0 -${M_PI/2} 0.0"/>
+</softkinetic_camera>
 </robot>

File: armadillo2_description/urdf/armadillo2_gazebo.xacro (robot description, xacro)
@@ -2,5 +2,5 @@
 <robot xmlns:xacro="http://www.ros.org/wiki/xacro" name="armadillo2_robot" description="ARMadillo2 Robot">
     <xacro:include filename="$(find armadillo2_description)/urdf/armadillo2.xacro" />
-    <xacro:include filename="$(find armadillo2_gazebo)/macros/intel_cam.xacro" />
+    <xacro:include filename="$(find armadillo2_gazebo)/macros/softkinetic_camera_ds325.xacro" />
     <xacro:arg name="kinect2" default="true"/>
     <xacro:arg name="kinect2_hz" default="30.0"/>
@@ -12,9 +12,8 @@
     <xacro:arg name="gps" default="true"/>
     <xacro:arg name="lidar" default="true"/>
-    <xacro:arg name="intel_cam" default="true"/>
-    <!-- intel_cam -->
-    <xacro:if value="$(arg intel_cam)">
-        <xacro:include filename="$(find armadillo2_gazebo)/macros/intel_cam.xacro" />
-        <xacro:intel_d435_gazebo name="camera" ros_topic="intel_cam"/>
+    <xacro:arg name="softkinetic" default="true"/>
+    <!-- softkinetic -->
+    <xacro:if value="$(arg softkinetic)">
+        <xacro:softkinetic_gazebo name="softkinetic_rgb" ros_topic="softkinetic"/>
     </xacro:if>
     <!-- kinect 2 -->

Commit message: Update armadillo2.xacro

File: armadillo2_description/urdf/armadillo2.xacro (robot description, xacro)
@@ -1,7 +1,7 @@
 <?xml version="1.0"?>
-<robot xmlns:xacro="http://www.ros.org/wiki/xacro" name="armadillo2_robot" description="ARMadillo2 Robot">
+<robot xmlns:xacro="http://www.ros.org/wiki/xacro" name="armadillo_robot" description="armadillo robot">
  <xacro:property name="M_PI" value="3.1415926535897931" />
- <xacro:property name="WHEEL_RADIUS" value="0.095" />
- <xacro:include filename="$(find armadillo2_description)/urdf/intel_d435.urdf"/>
+ <xacro:property name="WHEEL_RADIUS" value="0.1016" />
+ <xacro:include filename="$(find mobilican_description)/armadillo_2/urdf/intel_d435.urdf"/>
 <link name="base_footprint"/>
  <joint name="base_footprint_joint" type="fixed">
@@ -16,13 +16,14 @@
         xyz="-0.012353 0.000122 0.17716"
         rpy="0 0 0" />
-       <mass value="100.0"/>
-       <inertia
-        ixx="0.31639"
-        ixy="-9.1727E-05"
-        ixz="-0.093044"
-        iyy="0.17997"
-        iyz="5.3231E-05"
-        izz="0.16693" />
-    </inertial>
+       <mass
+        value="100" />
+        <inertia
+          ixx="0.31639"
+          ixy="-9.1727E-05"
+          ixz="-0.093044"
+          iyy="0.017997"
+          iyz="5.3231E-05"
+          izz="0.16693" />
+        </inertial>
     <visual>
       <origin
@@ -49,24 +50,4 @@
           </collision>
   </link>
-    <joint name="caster_front_left_joint" type="fixed">
-      <parent link="base_link"/>
-      <child link="caster_front_left_link"/>
-      <origin xyz="0.2 0.24 ${-WHEEL_RADIUS+0.0115+0.05+0.015}" rpy="${-M_PI/2} 0 0"/>
-    </joint>
-    <link name="caster_front_left_link">
-      <collision>
-        <geometry>
-          <cylinder length="0.0176" radius="0.05"/>
-        </geometry>
-        <origin rpy="0 0 0" xyz="0 0 0"/>
-      </collision>
-      <inertial>
-        <mass value="0.01" />
-        <origin xyz="0 0 0" />
-        <inertia ixx="0.001" ixy="0.0" ixz="0.0"
-                 iyy="0.001" iyz="0.0"
-                 izz="0.001" />
-      </inertial>
-    </link>
     <joint name="caster_back_left_joint" type="fixed">
       <parent link="base_link"/>
@@ -77,34 +58,18 @@
       <collision>
         <geometry>
-          <cylinder length="0.0176" radius="0.05"/>
+          <cylinder length="0.06" radius="0.05"/>
         </geometry>
-        <origin rpy="0 0 0" xyz="0 0 0"/>
+        <origin rpy="0 0 0" xyz="0 0 -0.03"/>
       </collision>
       <inertial>
-        <mass value="0.01" />
+        <mass value="0.0001" />
         <origin xyz="0 0 0" />
-        <inertia ixx="0.001" ixy="0.0" ixz="0.0"
-                 iyy="0.001" iyz="0.0"
-                 izz="0.001" />
-      </inertial>
-    </link>
-        <joint name="caster_front_right_joint" type="fixed">
-      <parent link="base_link"/>
-      <child link="caster_front_right_link"/>
-      <origin xyz="0.2 -0.24 ${-WHEEL_RADIUS+0.0115+0.05+0.015}" rpy="${-M_PI/2} 0 0"/>
-    </joint>
-    <link name="caster_front_right_link">
-      <collision>
-        <geometry>
-          <cylinder length="0.0176" radius="0.05"/>
-        </geometry>
-        <origin rpy="0 0 0" xyz="0 0 0"/>
-      </collision>
-      <inertial>
-        <mass value="0.01" />
-        <origin xyz="0 0 0" />
-        <inertia ixx="0.001" ixy="0.0" ixz="0.0"
-                 iyy="0.001" iyz="0.0"
-                 izz="0.001" />
+        <inertia
+        ixx="0.0069046"
+        ixy="-3.8717E-08"
+        ixz="2.0707E-07"
+        iyy="0.01"
+        iyz="-1.0124E-07"
+        izz="0.0069054" />
       </inertial>
     </link>
@@ -117,14 +82,18 @@
       <collision>
         <geometry>
-          <cylinder length="0.0176" radius="0.05"/>
+          <cylinder length="0.06" radius="0.05"/>
         </geometry>
-        <origin rpy="0 0 0" xyz="0 0 0"/>
+        <origin rpy="0 0 0" xyz="0 0 0.03"/>
       </collision>
       <inertial>
-        <mass value="0.01" />
+        <mass value="0.0001" />
         <origin xyz="0 0 0" />
-        <inertia ixx="0.001" ixy="0.0" ixz="0.0"
-                 iyy="0.001" iyz="0.0"
-                 izz="0.001" />
+        <inertia
+        ixx="0.0069046"
+        ixy="-3.8717E-08"
+        ixz="2.0707E-07"
+        iyy="0.01"
+        iyz="-1.0124E-07"
+        izz="0.0069054" />
       </inertial>
     </link>
@@ -136,10 +105,10 @@
         rpy="0 0 0" />
     <mass
-        value="1.8524" />
+        value="1.5" />
       <inertia
         ixx="0.0069046"
         ixy="-3.8717E-08"
         ixz="2.0707E-07"
-        iyy="0.013153"
+        iyy="0.01"
         iyz="-1.0124E-07"
         izz="0.0069054" />
@@ -164,5 +133,5 @@
         rpy="${M_PI/2} 0 0" />
       <geometry>
-      <cylinder  length="0.04" radius="${WHEEL_RADIUS}"/>
+      <cylinder  length="0.07" radius="${WHEEL_RADIUS}"/>
       </geometry>
     </collision>
@@ -191,10 +160,10 @@
         rpy="0 0 0" />
        <mass
-        value="1.8524" />
+        value="1.5" />
       <inertia
         ixx="0.0069046"
         ixy="-3.8717E-08"
         ixz="-2.0707E-07"
-        iyy="0.013153"
+        iyy="0.01"
         iyz="1.0124E-07"
         izz="0.0069054" />
@@ -219,5 +188,5 @@
         rpy="${M_PI/2} 0 0" />
       <geometry>
-      <cylinder  length="0.04" radius="${WHEEL_RADIUS}"/>
+      <cylinder  length="0.07" radius="${WHEEL_RADIUS}"/>
       </geometry>
     </collision>
@@ -241,4 +210,18 @@
  <link
     name="caster_left_link">
+     <inertial>
+      <origin
+        xyz="9.16610941069373E-06 -4.99540929455033E-06 8.06098359126817E-06"
+        rpy="0 0 0" />
+       <mass
+        value="20" />
+      <inertia
+        ixx="0.0069046"
+        ixy="-3.8717E-08"
+        ixz="-2.0707E-07"
+        iyy="0.01"
+        iyz="1.0124E-07"
+        izz="0.0069054" />
+    </inertial>
     <visual>
       <origin
@@ -301,4 +284,18 @@
   <link
     name="caster_right_link">
+      <inertial>
+      <origin
+        xyz="9.16610941069373E-06 -4.99540929455033E-06 8.06098359126817E-06"
+        rpy="0 0 0" />
+       <mass
+        value="20" />
+      <inertia
+        ixx="0.0069046"
+        ixy="-3.8717E-08"
+        ixz="-2.0707E-07"
+        iyy="0.01"
+        iyz="1.0124E-07"
+        izz="0.0069054" />
+    </inertial>
     <visual>
       <origin
@@ -336,12 +333,12 @@
         rpy="0 0 0" />
      <mass
-        value="0.035511" />
+        value="0.1" />
       <inertia
         ixx="0.09579"
         ixy="2.4285E-05"
         ixz="-0.0045097"
-        iyy="0.06807"
+        iyy="0.0001"
         iyz="-7.4938E-05"
-        izz="0.072852" />
+        izz="0.00032852" />
     </inertial>
     <visual>
@@ -373,5 +370,5 @@
         rpy="0 0 0" />
       <geometry>
-        <box size="0.09 0.5 0.8"/>
+        <box size="0.09 0.5 0.6"/>
       </geometry>
     </collision>
@@ -394,5 +391,5 @@
       effort="0.001"
       velocity="0.1" />
-<dynamics damping="0.1" friction="0"/>
+<!--<dynamics damping="0.1" friction="0"/>-->
   </joint>
   <link
@@ -403,5 +400,5 @@
         rpy="0 0 0" />
       <mass
-        value="0.003653" />
+        value="0.001" />
       <inertia
         ixx="3.6365E-05"
@@ -453,5 +450,5 @@
       effort="0.5"
       velocity="2" />
-<dynamics damping="0.1" friction="0"/>
+<!--<dynamics damping="0.1" friction="0"/>-->
   </joint>
   <link
@@ -462,5 +459,5 @@
         rpy="0 0 0" />
       <mass
-        value="0.00232" />
+        value="0.001" />
       <inertia
         ixx="0.00056403"
@@ -512,5 +509,5 @@
       effort="0.5"
       velocity="2" />
-<dynamics damping="0.1" friction="0"/>
+<!--<dynamics damping="0.1" friction="0"/>-->
   </joint>
   <link
@@ -521,5 +518,5 @@
         rpy="0 0 0" />
       <mass
-        value="0.00232" />
+        value="0.001" />
       <inertia
         ixx="0.00056403"
@@ -578,5 +575,5 @@
         rpy="0 0 0" />
       <mass
-        value="0.05" />
+        value="0.001" />
       <inertia
         ixx="0.00055596"
@@ -628,5 +625,5 @@
       upper="1.57"
       velocity="2.0" />
-<dynamics damping="0.1" friction="0"/>
+<!--<dynamics damping="0.1" friction="0"/>-->
   </joint>
   <link
@@ -637,5 +634,5 @@
         rpy="0 0 0" />
       <mass
-        value="0.05" />
+        value="0.001" />
       <inertia
         ixx="0.0043595"
@@ -687,5 +684,5 @@
       upper="1.95"
       velocity="2.0" />
-<dynamics damping="0.1" friction="0"/>
+<!--<dynamics damping="0.1" friction="0"/>-->
   </joint>
   <link
@@ -696,5 +693,5 @@
         rpy="0 0 0" />
       <mass
-        value="0.5" />
+        value="0.001" />
       <inertia
         ixx="0.00093237"
@@ -746,5 +743,5 @@
       upper="2.3522"
       velocity="2.0" />
-<dynamics damping="0.1" friction="0"/>
+<!--<dynamics damping="0.1" friction="0"/>-->
   </joint>
   <link
@@ -755,5 +752,5 @@
         rpy="0 0 0" />
       <mass
-        value="0.03" />
+        value="0.001" />
       <inertia
         ixx="0.00014092"
@@ -805,5 +802,5 @@
       upper="1.57"
       velocity="2.0" />
-<dynamics damping="0.1" friction="0"/>
+<!--<dynamics damping="0.1" friction="0"/>-->
   </joint>
   <link
@@ -814,5 +811,5 @@
         rpy="0 0 0" />
       <mass
-        value="0.03" />
+        value="0.001" />
       <inertia
         ixx="0.00018198"
@@ -864,5 +861,5 @@
       upper="1.57"
       velocity="2.0" />
-<dynamics damping="0.1" friction="0"/>
+<!--<dynamics damping="0.1" friction="0"/>-->
   </joint>
   <link
@@ -873,5 +870,5 @@
         rpy="0 0 0" />
       <mass
-        value="0.03" />
+        value="0.001" />
       <inertia
         ixx="4.4099E-05"
@@ -923,5 +920,5 @@
       upper="3.14"
       velocity="2.0" />
-<dynamics damping="0.5" friction="0.5"/>
+<!--<dynamics damping="0.5" friction="0.5"/>-->
   </joint>
   <link name="gripper_link"/>
@@ -938,5 +935,5 @@
         rpy="0 0 0" />
       <mass
-        value="0.01" />
+        value="0.001" />
       <inertia
         ixx="1.4683E-05"
@@ -988,5 +985,5 @@
       upper="1.57"
       velocity="0.1" />
-<dynamics damping="0.5" friction="0.5"/>
+<!--<dynamics damping="0.5" friction="0.5"/>-->
   </joint>
   <link
@@ -997,5 +994,5 @@
         rpy="0 0 0" />
       <mass
-        value="0.01" />
+        value="0.001" />
       <inertia
         ixx="1.4683E-05"
@@ -1047,59 +1044,6 @@
       upper="1.57"
       velocity="0.1" />
-<dynamics damping="0.5" friction="0.5"/>
-  </joint>
- <!-- <joint
-    name="intel_d435_joint"
-    type="fixed">
-    <origin
-      xyz="0 0.0143 -0.049"
-      rpy="-3.1416 0 1.5708" />
-    <parent
-      link="wrist_link" />
-    <child
-      link="intel_d435_link" />
-    <axis
-      xyz="0 0 0" />
-    </joint>-->
-  <!--<link
-    name="intel_d435_link">
-    <inertial>
-      <origin
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