Commit message: removed ric_interface. with catkin_ignore

File: armadillo2_description/urdf/armadillo2_gazebo.xacro (robot description, xacro)
@@ -1,6 +1,5 @@
 <?xml version="1.0"?>
-<robot xmlns:xacro="http://www.ros.org/wiki/xacro" name="armadillo2_robot" description="ARMadillo2 Robot">
-    <xacro:include filename="$(find armadillo2_description)/urdf/armadillo2.xacro" />
-    <xacro:include filename="$(find armadillo2_gazebo)/macros/softkinetic_camera_ds325.xacro" />
+<robot xmlns:xacro="http://www.ros.org/wiki/xacro" name="armadillo2_robot" description="armadillo2 robot">
+  <xacro:include filename="$(find armadillo2_description)/urdf/armadillo2.xacro" />
     <xacro:arg name="kinect2" default="true"/>
     <xacro:arg name="kinect2_hz" default="30.0"/>
@@ -12,8 +11,24 @@
     <xacro:arg name="gps" default="true"/>
     <xacro:arg name="lidar" default="true"/>
-    <xacro:arg name="softkinetic" default="true"/>
-    <!-- softkinetic -->
-    <xacro:if value="$(arg softkinetic)">
-        <xacro:softkinetic_gazebo name="softkinetic_rgb" ros_topic="softkinetic"/>
+    <xacro:arg name="intel_cam" default="true"/>
+    <!-- intel_cam -->
+    <xacro:if value="$(arg intel_cam)">
+        <xacro:include filename="$(find armadillo2_gazebo)/macros/intel_cam.xacro" />
+        <xacro:DepthCam name="intel_cam"
+                        link="camera_link"
+                        optical_frame="camera_depth_optical_frame"
+                        horizontal_fov="1.592"
+                        img_width="1280"
+                        img_height="800"
+                        img_format="B8G8R8"
+                        clip_near="0.1"
+                        clip_far="100"
+                        update_rate="10.0"
+                        image_topic="color/image_raw"
+                        depth_topic="depth/color/image_raw"
+                        cloud_topic="depth/color/points"
+                        info_topic="color/camera_info"
+                        depth_info_topic="depth/camera_info"
+                        pointcloud_cuttoff="0.2" />
     </xacro:if>
     <!-- kinect 2 -->
@@ -28,11 +43,30 @@
     <xacro:if value="$(arg urf)">
         <xacro:include filename="$(find armadillo2_gazebo)/macros/urf.xacro" />
-        <xacro:urf name="front" link="front_urf_link" topic="URF/front" fov="${10.0*M_PI/180.0}" min="0.2" max="5.0"/>
+        <xacro:urf name="front" link="front_urf_link" topic="urf/front" fov="${10.0*M_PI/180.0}" min="0.3" max="5.0" update_rate="10"/>
     </xacro:if>
     <!-- hokuyo  utm-30lx -->
     <xacro:if value="$(arg lidar)">
-        <xacro:include filename="$(find armadillo2_gazebo)/macros/hokuyo.xacro" />
-        <xacro:lidar link="laser_link" topic="scan" samples="720" resolution="1" min_angle="-1.5707963" max_angle="1.5707963" range_min="0.1" range_max="30" range_resolution="0.03" />
-    </xacro:if>
+        <xacro:include filename="$(find armadillo2_gazebo)/macros/lidar.xacro" />
+        <xacro:lidar name="lidar"
+                     link="laser_link"
+                     topic="scan"
+                     update_rate="10"
+                     samples="720"
+                     resolution="1"
+                     min_angle="-1.5707"
+                     max_angle="1.5707"
+                     range_min="0.1"
+                     range_max="30.0"
+                     range_resolution="0.01" />
+    </xacro:if>
+    <!-- sim ODOM -->
+    <!-- <gazebo>
+      <plugin name="sim_odom" filename="libgazebo_ros_p3d.so">
+        <frameName>map</frameName>
+        <bodyName>base_footprint</bodyName>
+        <topicName>sim_odom</topicName>
+        <updateRate>10.0</updateRate>
+      </plugin>
+    </gazebo> -->
     <!-- GPS   -->
     <xacro:if value="$(arg gps)">
@@ -47,4 +81,5 @@
     <gazebo>
         <plugin name="gazebo_ros_control" filename="libgazebo_ros_control.so">
+            <!-- <legacyModeNS>true</legacyModeNS> -->
             <robotSimType>gazebo_ros_control/Armadillo2RobotHWSim</robotSimType>
         </plugin>
@@ -54,7 +89,7 @@
             <arm>
                 <arm_name>arm</arm_name>
-                <palm_link> wrist_link  </palm_link>
-                <gripper_link> left_finger_link </gripper_link>
-                <gripper_link> right_finger_link </gripper_link>
+                <palm_link>wrist_link</palm_link>
+                <gripper_link>left_finger_link</gripper_link>
+                <gripper_link>right_finger_link</gripper_link>
             </arm>
             <forces_angle_tolerance>100</forces_angle_tolerance>
@@ -67,25 +102,54 @@
         </plugin>
     </gazebo>
-    <gazebo reference="left_finger_link">
-        <kp>1000000.0</kp>
-        <kd>1.0</kd>
-        <mu1>1.0</mu1>
-        <mu2>1.0</mu2>
-        <fdir1>0 0 1</fdir1>
-        <maxVel>1.0</maxVel>
-        <minDepth>0.001</minDepth>
-    </gazebo>
-    <gazebo reference="left_finger_joint">
+    <transmission name="left_wheel_joint_trans">
+        <type>transmission_interface/SimpleTransmission</type>
+        <joint name="left_wheel_joint">
+            <hardwareInterface>hardware_interface/VelocityJointInterface</hardwareInterface>
+        </joint>
+        <actuator name="left_wheel_joint_motor">
+            <mechanicalReduction>1</mechanicalReduction>
+        </actuator>
+    </transmission>
+    <transmission name="right_wheel_joint_trans">
+        <type>transmission_interface/SimpleTransmission</type>
+        <joint name="right_wheel_joint">
+            <hardwareInterface>hardware_interface/VelocityJointInterface</hardwareInterface>
+        </joint>
+        <actuator name="right_wheel_joint_motor">
+            <mechanicalReduction>1</mechanicalReduction>
+        </actuator>
+    </transmission>
+    <transmission name="torso_joint_trans">
+        <type>transmission_interface/SimpleTransmission</type>
+        <joint name="torso_joint">
+            <hardwareInterface>hardware_interface/EffortJointInterface</hardwareInterface>
+        </joint>
+        <actuator name="torso_joint_motor">
+            <mechanicalReduction>1</mechanicalReduction>
+        </actuator>
+    </transmission>
+    <transmission name="head_pan_joint_trans">
+        <type>transmission_interface/SimpleTransmission</type>
+        <joint name="head_pan_joint">
+            <hardwareInterface>hardware_interface/PositionJointInterface</hardwareInterface>
+        </joint>
+        <actuator name="head_pan_joint_motor">
+            <mechanicalReduction>1</mechanicalReduction>
+        </actuator>
+    </transmission>
+    <transmission name="head_tilt_joint_trans">
+        <type>transmission_interface/SimpleTransmission</type>
+        <joint name="head_tilt_joint">
+            <hardwareInterface>hardware_interface/PositionJointInterface</hardwareInterface>
+        </joint>
+        <actuator name="head_tilt_joint_motor">
+            <mechanicalReduction>1</mechanicalReduction>
+        </actuator>
+    </transmission>
+    <xacro:property name="mu1" value="2.0" />
+    <xacro:property name="mu2" value="2.0" />
+     <gazebo reference="left_finger_joint">
         <implicitSpringDamper>1</implicitSpringDamper>
         <provideFeedback>1</provideFeedback>
-    </gazebo>
-    <gazebo reference="right_finger_link">
-        <kp>1000000.0</kp>
-        <kd>1.0</kd>
-        <mu1>1.0</mu1>
-        <mu2>1.0</mu2>
-        <fdir1>0 0 1</fdir1>
-        <maxVel>1.0</maxVel>
-        <minDepth>0.001</minDepth>
     </gazebo>
     <gazebo reference="right_finger_joint">
@@ -93,105 +157,75 @@
         <provideFeedback>1</provideFeedback>
     </gazebo>
-    <transmission name="left_wheel_joint_trans">
-        <type>transmission_interface/SimpleTransmission</type>
-        <joint name="left_wheel_joint">
-            <hardwareInterface>VelocityJointInterface</hardwareInterface>
-        </joint>
-        <actuator name="left_wheel_joint_motor">
-            <mechanicalReduction>1</mechanicalReduction>
-        </actuator>
-    </transmission>
-    <transmission name="right_wheel_joint_trans">
-        <type>transmission_interface/SimpleTransmission</type>
-        <joint name="right_wheel_joint">
-            <hardwareInterface>VelocityJointInterface</hardwareInterface>
-        </joint>
-        <actuator name="right_wheel_joint_motor">
-            <mechanicalReduction>1</mechanicalReduction>
-        </actuator>
-    </transmission>
-    <transmission name="torso_joint_trans">
-        <type>transmission_interface/SimpleTransmission</type>
-        <joint name="torso_joint">
-            <hardwareInterface>PositionJointInterface</hardwareInterface>
-        </joint>
-        <actuator name="torso_joint_motor">
-            <mechanicalReduction>1</mechanicalReduction>
-        </actuator>
-    </transmission>
-    <transmission name="head_pan_joint_trans">
-        <type>transmission_interface/SimpleTransmission</type>
-        <joint name="head_pan_joint">
-            <hardwareInterface>PositionJointInterface</hardwareInterface>
-        </joint>
-        <actuator name="head_pan_joint_motor">
-            <mechanicalReduction>1</mechanicalReduction>
-        </actuator>
-    </transmission>
-    <transmission name="head_tilt_joint_trans">
-        <type>transmission_interface/SimpleTransmission</type>
-        <joint name="head_tilt_joint">
-            <hardwareInterface>PositionJointInterface</hardwareInterface>
-        </joint>
-        <actuator name="head_tilt_joint_motor">
-            <mechanicalReduction>1</mechanicalReduction>
-        </actuator>
-    </transmission>
+    <gazebo reference="right_finger_link">
+        <!-- kp and kd for rubber -->
+        <!-- <kp>1000000.0</kp>
+        <kd>100.0</kd> -->
+        <mu1>1000</mu1>
+        <mu2>1000</mu2>
+        <fdir1>1 0 0</fdir1>
+        <maxVel>1.0</maxVel>
+        <minDepth>0.001</minDepth>
+    </gazebo>
+    <gazebo reference="left_finger_link">
+        <!-- kp and kd for rubber -->
+        <!-- <kp>1000000.0</kp>
+        <kd>100.0</kd> -->
+        <mu1>1000</mu1>
+        <mu2>1000</mu2>
+        <fdir1>1 0 0</fdir1>
+        <maxVel>1.0</maxVel>
+        <minDepth>0.001</minDepth>
+    </gazebo>
     <gazebo reference="left_wheel_link">
-        <mu1>2.0</mu1>
-        <mu2>2.0</mu2>
+        <!-- kp and kd for rubber -->
         <kp>1000000.0</kp>
         <kd>100.0</kd>
-        <minDepth>0.001</minDepth>
-        <maxVel>1.0</maxVel>
+        <mu1>${mu1}</mu1>
+        <mu2>${mu2}</mu2>
+        <fdir1>1 0 0</fdir1>
+        <maxVel>1.0</maxVel>
+        <minDepth>0.001</minDepth>
+        <material>Gazebo/DarkGrey</material>
     </gazebo>
     <gazebo reference="right_wheel_link">
-        <mu1>2.0</mu1>
-        <mu2>2.0</mu2>
+        <!-- kp and kd for rubber -->
         <kp>1000000.0</kp>
         <kd>100.0</kd>
-        <minDepth>0.001</minDepth>
-        <maxVel>1.0</maxVel>
-    </gazebo>
-    <gazebo reference="caster_front_right_link">
+        <mu1>${mu1}</mu1>
+        <mu2>${mu2}</mu2>
+        <fdir1>1 0 0</fdir1>
+        <maxVel>1.0</maxVel>
+        <minDepth>0.001</minDepth>
+        <material>Gazebo/DarkGrey</material>
+    </gazebo>
+    <gazebo reference="caster_left_link">
+        <!-- kp and kd for rubber -->
+        <kp>1000000.0</kp>
+        <kd>1000.0</kd>
         <mu1>0.0</mu1>
         <mu2>0.0</mu2>
+        <fdir1>1 0 0</fdir1>
+        <maxVel>1.0</maxVel>
+        <minDepth>0.001</minDepth>
+        <material>Gazebo/DarkGrey</material>
+    </gazebo>
+    <gazebo reference="caster_right_link">
+    <!-- kp and kd for rubber -->
         <kp>1000000.0</kp>
-        <kd>100.0</kd>
-        <minDepth>0.001</minDepth>
-        <maxVel>1.0</maxVel>
-    </gazebo>
-    <gazebo reference="caster_back_right_link">
+        <kd>1000.0</kd>
         <mu1>0.0</mu1>
         <mu2>0.0</mu2>
-        <kp>1000000.0</kp>
-        <kd>100.0</kd>
-        <minDepth>0.001</minDepth>
-        <maxVel>1.0</maxVel>
-    </gazebo>
-        <gazebo reference="caster_front_left_link">
-        <mu1>0.0</mu1>
-        <mu2>0.0</mu2>
-        <kp>1000000.0</kp>
-        <kd>100.0</kd>
-        <minDepth>0.001</minDepth>
-        <maxVel>1.0</maxVel>
-    </gazebo>
-    <gazebo reference="caster_back_left_link">
-        <mu1>0.0</mu1>
-        <mu2>0.0</mu2>
-        <kp>1000000.0</kp>
-        <kd>100.0</kd>
-        <minDepth>0.001</minDepth>
-        <maxVel>1.0</maxVel>
+        <fdir1>1 0 0</fdir1>
+        <maxVel>1.0</maxVel>
+        <minDepth>0.001</minDepth>
+        <material>Gazebo/DarkGrey</material>
     </gazebo>
     <gazebo reference="base_link">
-        <mu1>0.3</mu1>
-        <mu2>0.3</mu2>
+        <material>Gazebo/Grey</material>
     </gazebo>
     <transmission name="rotation1_joint_trans">
         <type>transmission_interface/SimpleTransmission</type>
         <joint name="rotation1_joint">
-            <hardwareInterface>PosVelJointInterface</hardwareInterface>
+            <hardwareInterface>hardware_interface/PosVelJointInterface</hardwareInterface>
         </joint>
         <actuator name="rotation1_joint_motor">
@@ -202,5 +236,5 @@
         <type>transmission_interface/SimpleTransmission</type>
         <joint name="shoulder1_joint">
-            <hardwareInterface>PosVelJointInterface</hardwareInterface>
+            <hardwareInterface>hardware_interface/PosVelJointInterface</hardwareInterface>
         </joint>
         <actuator name="shoulder1_joint_motor">
@@ -211,5 +245,5 @@
         <type>transmission_interface/SimpleTransmission</type>
         <joint name="shoulder2_joint">
-            <hardwareInterface>PosVelJointInterface</hardwareInterface>
+            <hardwareInterface>hardware_interface/PosVelJointInterface</hardwareInterface>
         </joint>
         <actuator name="shoulder2_joint_motor">
@@ -220,5 +254,5 @@
         <type>transmission_interface/SimpleTransmission</type>
         <joint name="rotation2_joint">
-            <hardwareInterface>PosVelJointInterface</hardwareInterface>
+            <hardwareInterface>hardware_interface/PosVelJointInterface</hardwareInterface>
         </joint>
         <actuator name="rotation2_joint_motor">
@@ -229,5 +263,5 @@
         <type>transmission_interface/SimpleTransmission</type>
         <joint name="shoulder3_joint">
-            <hardwareInterface>PosVelJointInterface</hardwareInterface>
+            <hardwareInterface>hardware_interface/PosVelJointInterface</hardwareInterface>
         </joint>
         <actuator name="shoulder3_joint_motor">
@@ -238,5 +272,5 @@
         <type>transmission_interface/SimpleTransmission</type>
         <joint name="wrist_joint">
-            <hardwareInterface>PosVelJointInterface</hardwareInterface>
+            <hardwareInterface>hardware_interface/PosVelJointInterface</hardwareInterface>
         </joint>
         <actuator name="wrist_joint_motor">
@@ -247,5 +281,5 @@
         <type>transmission_interface/SimpleTransmission</type>
         <joint name="left_finger_joint">
-            <hardwareInterface>PosVelJointInterface</hardwareInterface>
+            <hardwareInterface>hardware_interface/PosVelJointInterface</hardwareInterface>
         </joint>
         <actuator name="left_finger_joint_motor">
@@ -256,5 +290,5 @@
         <type>transmission_interface/SimpleTransmission</type>
         <joint name="right_finger_joint">
-            <hardwareInterface>PosVelJointInterface</hardwareInterface>
+            <hardwareInterface>hardware_interface/PosVelJointInterface</hardwareInterface>
         </joint>
         <actuator name="right_finger_joint_motor">
@@ -262,3 +296,51 @@
         </actuator>
     </transmission>
+    <!-- Link1 -->
+  <gazebo reference="rotation1_link">
+    <mu1>0.2</mu1>
+    <mu2>0.2</mu2>
+    <material>Gazebo/Grey</material>
+  </gazebo>
+  <!-- Link2 -->
+  <gazebo reference="shoulder1_link">
+    <mu1>0.2</mu1>
+    <mu2>0.2</mu2>
+    <material>Gazebo/Grey</material>
+  </gazebo>
+  <!-- Link3 -->
+  <gazebo reference="shoulder2_link">
+    <mu1>0.2</mu1>
+    <mu2>0.2</mu2>
+    <material>Gazebo/Grey</material>
+  </gazebo>
+  <!-- Link4 -->
+  <gazebo reference="rotation2_link">
+    <mu1>0.2</mu1>
+    <mu2>0.2</mu2>
+    <material>Gazebo/Grey</material>
+  </gazebo>
+  <!-- Link5 -->
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
Commit message: removed change notifiers

File: armadillo2_description/urdf/armadillo2.xacro (robot description, xacro)
@@ -230,5 +230,5 @@
     </collision>
   </link>
-  <joint name="torso_joint" type="prismatic"> <!--fixed YAMYAIR-->
+  <joint name="torso_joint" type="prismatic">
     <origin xyz="0 0 0" rpy="0 0 0" />
     <parent link="base_link" />
