Commit message: renaming files

File: armadillo_description/urdf/armadillo.xacro (robot description, xacro)
@@ -1,7 +1,7 @@
 <?xml version="1.0"?>
-<robot xmlns:xacro="http://www.ros.org/wiki/xacro" name="armadillo2_robot" description="ARMadillo2 Robot">
+<robot xmlns:xacro="http://www.ros.org/wiki/xacro" name="armadillo_robot" description="armadillo robot">
  <xacro:property name="M_PI" value="3.1415926535897931" />
  <xacro:property name="WHEEL_RADIUS" value="0.095" />
- <xacro:include filename="$(find armadillo2_description)/urdf/intel_d435.urdf"/>
+ <xacro:include filename="$(find armadillo_description)/urdf/intel_d435.urdf"/>
 <link name="base_footprint"/>
  <joint name="base_footprint_joint" type="fixed">
@@ -31,5 +31,5 @@
       <geometry>
         <mesh
-          filename="package://armadillo2_description/mesh/base_link.STL" />
+          filename="package://armadillo_description/mesh/base_link.STL" />
       </geometry>
       <material
@@ -45,5 +45,5 @@
       <geometry>
         <mesh
-          filename="package://armadillo2_description/mesh/base_link.STL" />
+          filename="package://armadillo_description/mesh/base_link.STL" />
       </geometry>
           </collision>
@@ -151,5 +151,5 @@
       <geometry>
         <mesh
-          filename="package://armadillo2_description/mesh/left_wheel_link.STL" />
+          filename="package://armadillo_description/mesh/left_wheel_link.STL" />
       </geometry>
       <material
@@ -206,5 +206,5 @@
       <geometry>
         <mesh
-          filename="package://armadillo2_description/mesh/right_wheel_link.STL" />
+          filename="package://armadillo_description/mesh/right_wheel_link.STL" />
       </geometry>
       <material
@@ -247,5 +247,5 @@
       <geometry>
         <mesh
-          filename="package://armadillo2_description/mesh/caster_left_link.STL" />
+          filename="package://armadillo_description/mesh/caster_left_link.STL" />
       </geometry>
       <material
@@ -307,5 +307,5 @@
       <geometry>
         <mesh
-          filename="package://armadillo2_description/mesh/caster_right_link.STL" />
+          filename="package://armadillo_description/mesh/caster_right_link.STL" />
       </geometry>
       <material
@@ -351,5 +351,5 @@
       <geometry>
         <mesh
-          filename="package://armadillo2_description/mesh/torso_link.STL" />
+          filename="package://armadillo_description/mesh/torso_link.STL" />
       </geometry>
       <material
@@ -365,5 +365,5 @@
       <geometry>
         <mesh
-          filename="package://armadillo2_description/mesh/torso_link.STL" />
+          filename="package://armadillo_description/mesh/torso_link.STL" />
       </geometry>
     </collision>
@@ -418,5 +418,5 @@
       <geometry>
         <mesh
-          filename="package://armadillo2_description/mesh/head_pan_link.STL" />
+          filename="package://armadillo_description/mesh/head_pan_link.STL" />
       </geometry>
       <material
@@ -432,5 +432,5 @@
       <geometry>
         <mesh
-          filename="package://armadillo2_description/mesh/head_pan_link.STL" />
+          filename="package://armadillo_description/mesh/head_pan_link.STL" />
       </geometry>
     </collision>
@@ -477,5 +477,5 @@
       <geometry>
         <mesh
-          filename="package://armadillo2_description/mesh/head_tilt_link.STL" />
+          filename="package://armadillo_description/mesh/head_tilt_link.STL" />
       </geometry>
       <material
@@ -491,5 +491,5 @@
       <geometry>
         <mesh
-          filename="package://armadillo2_description/mesh/head_tilt_link.STL" />
+          filename="package://armadillo_description/mesh/head_tilt_link.STL" />
       </geometry>
     </collision>
@@ -593,5 +593,5 @@
       <geometry>
         <mesh
-          filename="package://armadillo2_description/mesh/rotation1_link.STL" />
+          filename="package://armadillo_description/mesh/rotation1_link.STL" />
       </geometry>
       <material
@@ -607,5 +607,5 @@
       <geometry>
         <mesh
-          filename="package://armadillo2_description/mesh/rotation1_link.STL" />
+          filename="package://armadillo_description/mesh/rotation1_link.STL" />
       </geometry>
     </collision>
@@ -652,5 +652,5 @@
       <geometry>
         <mesh
-          filename="package://armadillo2_description/mesh/shoulder1_link.STL" />
+          filename="package://armadillo_description/mesh/shoulder1_link.STL" />
       </geometry>
       <material
@@ -666,5 +666,5 @@
       <geometry>
         <mesh
-          filename="package://armadillo2_description/mesh/shoulder1_link.STL" />
+          filename="package://armadillo_description/mesh/shoulder1_link.STL" />
       </geometry>
     </collision>
@@ -711,5 +711,5 @@
       <geometry>
         <mesh
-          filename="package://armadillo2_description/mesh/shoulder2_link.STL" />
+          filename="package://armadillo_description/mesh/shoulder2_link.STL" />
       </geometry>
       <material
@@ -725,5 +725,5 @@
       <geometry>
         <mesh
-          filename="package://armadillo2_description/mesh/shoulder2_link.STL" />
+          filename="package://armadillo_description/mesh/shoulder2_link.STL" />
       </geometry>
     </collision>
@@ -770,5 +770,5 @@
       <geometry>
         <mesh
-          filename="package://armadillo2_description/mesh/rotation2_link.STL" />
+          filename="package://armadillo_description/mesh/rotation2_link.STL" />
       </geometry>
       <material
@@ -784,5 +784,5 @@
       <geometry>
         <mesh
-          filename="package://armadillo2_description/mesh/rotation2_link.STL" />
+          filename="package://armadillo_description/mesh/rotation2_link.STL" />
       </geometry>
     </collision>
@@ -829,5 +829,5 @@
       <geometry>
         <mesh
-          filename="package://armadillo2_description/mesh/shoulder3_link.STL" />
+          filename="package://armadillo_description/mesh/shoulder3_link.STL" />
       </geometry>
       <material
@@ -843,5 +843,5 @@
       <geometry>
         <mesh
-          filename="package://armadillo2_description/mesh/shoulder3_link.STL" />
+          filename="package://armadillo_description/mesh/shoulder3_link.STL" />
       </geometry>
     </collision>
@@ -888,5 +888,5 @@
       <geometry>
         <mesh
-          filename="package://armadillo2_description/mesh/wrist_link.STL" />
+          filename="package://armadillo_description/mesh/wrist_link.STL" />
       </geometry>
       <material
@@ -902,5 +902,5 @@
       <geometry>
         <mesh
-          filename="package://armadillo2_description/mesh/wrist_link.STL" />
+          filename="package://armadillo_description/mesh/wrist_link.STL" />
       </geometry>
     </collision>
@@ -953,5 +953,5 @@
       <geometry>
         <mesh
-          filename="package://armadillo2_description/mesh/left_finger_link.STL" />
+          filename="package://armadillo_description/mesh/left_finger_link.STL" />
       </geometry>
       <material
@@ -967,5 +967,5 @@
       <geometry>
         <mesh
-          filename="package://armadillo2_description/mesh/left_finger_link.STL" />
+          filename="package://armadillo_description/mesh/left_finger_link.STL" />
       </geometry>
     </collision>
@@ -1012,5 +1012,5 @@
       <geometry>
         <mesh
-          filename="package://armadillo2_description/mesh/right_finger_link.STL" />
+          filename="package://armadillo_description/mesh/right_finger_link.STL" />
       </geometry>
       <material
@@ -1026,5 +1026,5 @@
       <geometry>
         <mesh
-          filename="package://armadillo2_description/mesh/right_finger_link.STL" />
+          filename="package://armadillo_description/mesh/right_finger_link.STL" />
       </geometry>
     </collision>
@@ -1084,5 +1084,5 @@
       <geometry>
         <mesh
-          filename="package://armadillo2_description/mesh/intel_d435.STL" />
+          filename="package://armadillo_description/mesh/intel_d435.STL" />
       </geometry>
       <material
@@ -1098,5 +1098,5 @@
       <geometry>
         <mesh
-          filename="package://armadillo2_description/mesh/intel_d435.STL" />
+          filename="package://armadillo_description/mesh/intel_d435.STL" />
       </geometry>
     </collision>

File: armadillo_description/urdf/armadillo_gazebo.xacro (robot description, xacro)
@@ -1,6 +1,6 @@
 <?xml version="1.0"?>
-<robot xmlns:xacro="http://www.ros.org/wiki/xacro" name="armadillo2_robot" description="ARMadillo2 Robot">
-    <xacro:include filename="$(find armadillo2_description)/urdf/armadillo2.xacro" />
-    <xacro:include filename="$(find armadillo2_gazebo)/macros/intel_cam.xacro" />
+<robot xmlns:xacro="http://www.ros.org/wiki/xacro" name="armadillo_robot" description="armadillo robot">
+    <xacro:include filename="$(find armadillo_description)/urdf/armadillo.xacro" />
+    <xacro:include filename="$(find armadillo_gazebo)/macros/intel_cam.xacro" />
     <xacro:arg name="kinect2" default="true"/>
     <xacro:arg name="kinect2_hz" default="30.0"/>
@@ -15,5 +15,5 @@
     <!-- intel_cam -->
     <xacro:if value="$(arg intel_cam)">
-        <xacro:include filename="$(find armadillo2_gazebo)/macros/intel_cam.xacro" />
+        <xacro:include filename="$(find armadillo_gazebo)/macros/intel_cam.xacro" />
         <xacro:intel_d435_gazebo name="camera" ros_topic="intel_cam"/>
     </xacro:if>
@@ -24,29 +24,29 @@
         <xacro:property name="kinect2_qhd" value="$(arg kinect2_qhd)"/>
         <xacro:property name="kinect2_sd" value="$(arg kinect2_sd)"/>
-        <xacro:include filename="$(find armadillo2_gazebo)/macros/kinect2.xacro" />
+        <xacro:include filename="$(find armadillo_gazebo)/macros/kinect2.xacro" />
     </xacro:if>
     <!-- Sonars -->
     <xacro:if value="$(arg urf)">
-        <xacro:include filename="$(find armadillo2_gazebo)/macros/urf.xacro" />
+        <xacro:include filename="$(find armadillo_gazebo)/macros/urf.xacro" />
         <xacro:urf name="front" link="front_urf_link" topic="URF/front" fov="${10.0*M_PI/180.0}" min="0.2" max="5.0"/>
     </xacro:if>
     <!-- hokuyo  utm-30lx -->
     <xacro:if value="$(arg lidar)">
-        <xacro:include filename="$(find armadillo2_gazebo)/macros/hokuyo.xacro" />
+        <xacro:include filename="$(find armadillo_gazebo)/macros/hokuyo.xacro" />
         <xacro:lidar link="laser_link" topic="scan" samples="720" resolution="1" min_angle="-1.5707963" max_angle="1.5707963" range_min="0.1" range_max="30" range_resolution="0.03" />
     </xacro:if>
     <!-- GPS   -->
     <xacro:if value="$(arg gps)">
-        <xacro:include filename="$(find armadillo2_gazebo)/macros/gps.xacro" />
+        <xacro:include filename="$(find armadillo_gazebo)/macros/gps.xacro" />
         <xacro:gps link="base_link" hz="5" topic="GPS" lat="31.262218" long="34.80146100" alt="298"/>
     </xacro:if>
     <!-- IMU   -->
     <xacro:if value="$(arg imu)">
-        <xacro:include filename="$(find armadillo2_gazebo)/macros/imu.xacro" />
+        <xacro:include filename="$(find armadillo_gazebo)/macros/imu.xacro" />
         <xacro:imu link="base_link" hz="50" topic="IMU" />
     </xacro:if>
     <gazebo>
         <plugin name="gazebo_ros_control" filename="libgazebo_ros_control.so">
-            <robotSimType>gazebo_ros_control/Armadillo2RobotHWSim</robotSimType>
+            <robotSimType>gazebo_ros_control/ArmadilloRobotHWSim</robotSimType>
         </plugin>
     </gazebo>

File: armadillo_description/urdf/intel_d435.urdf (robot description, URDF)
Before this commit: robot intel_d435, 9 links, 8 joints
Links:
- link camera_link: geometry collision mesh filename=package://armadillo_description/mesh/intel_d435.STL; visual mesh filename=package://armadillo_description/mesh/intel_d435.STL

Commit message: reduced upper body masses and enlarge wheels collisions

File: armadillo_description/urdf/armadillo.xacro (robot description, xacro)
@@ -77,7 +77,7 @@
       <collision>
         <geometry>
-          <cylinder length="0.0176" radius="0.05"/>
+          <cylinder length="0.06" radius="0.05"/>
         </geometry>
-        <origin rpy="0 0 0" xyz="0 0 0"/>
+        <origin rpy="0 0 0" xyz="0 0 -0.03"/>
       </collision>
       <inertial>
@@ -117,7 +117,7 @@
       <collision>
         <geometry>
-          <cylinder length="0.0176" radius="0.05"/>
+          <cylinder length="0.06" radius="0.05"/>
         </geometry>
-        <origin rpy="0 0 0" xyz="0 0 0"/>
+        <origin rpy="0 0 0" xyz="0 0 0.03"/>
       </collision>
       <inertial>
@@ -135,5 +135,5 @@
         xyz="9.16610941069373E-06 4.59070539915452E-09 8.0609835912647E-06"
         rpy="0 0 0" />
-    <mass
+   <mass
         value="1.8524" />
       <inertia
@@ -164,5 +164,5 @@
         rpy="${M_PI/2} 0 0" />
       <geometry>
-      <cylinder  length="0.04" radius="${WHEEL_RADIUS}"/>
+      <cylinder  length="0.07" radius="${WHEEL_RADIUS}"/>
       </geometry>
     </collision>
@@ -190,5 +190,5 @@
         xyz="9.16610941069373E-06 -4.99540929455033E-06 8.06098359126817E-06"
         rpy="0 0 0" />
-       <mass
+        <mass
         value="1.8524" />
       <inertia
@@ -219,5 +219,5 @@
         rpy="${M_PI/2} 0 0" />
       <geometry>
-      <cylinder  length="0.04" radius="${WHEEL_RADIUS}"/>
+      <cylinder  length="0.07" radius="${WHEEL_RADIUS}"/>
       </geometry>
     </collision>
@@ -336,5 +336,5 @@
         rpy="0 0 0" />
      <mass
-        value="0.035511" />
+        value="0.001" />
       <inertia
         ixx="0.09579"
@@ -403,5 +403,5 @@
         rpy="0 0 0" />
       <mass
-        value="0.003653" />
+        value="0.001" />
       <inertia
         ixx="3.6365E-05"
@@ -462,5 +462,5 @@
         rpy="0 0 0" />
       <mass
-        value="0.00232" />
+        value="0.001" />
       <inertia
         ixx="0.00056403"
@@ -521,5 +521,5 @@
         rpy="0 0 0" />
       <mass
-        value="0.00232" />
+        value="0.001" />
       <inertia
         ixx="0.00056403"
@@ -578,12 +578,12 @@
         rpy="0 0 0" />
       <mass
-        value="0.05" />
-      <inertia
-        ixx="0.00055596"
-        ixy="9.2522E-12"
-        ixz="9.2226E-12"
-        iyy="0.00016945"
-        iyz="6.1918E-06"
-        izz="0.00055286" />
+        value="0.001" />
+      <inertia
+        ixx="0.0043595"
+        ixy="-3.1405E-06"
+        ixz="0.00053636"
+        iyy="0.0041046"
+        iyz="-5.2275E-05"
+        izz="0.00081871" />
     </inertial>
     <visual>
@@ -637,5 +637,5 @@
         rpy="0 0 0" />
       <mass
-        value="0.05" />
+        value="0.001" />
       <inertia
         ixx="0.0043595"
@@ -696,5 +696,5 @@
         rpy="0 0 0" />
       <mass
-        value="0.5" />
+        value="0.001" />
       <inertia
         ixx="0.00093237"
@@ -754,6 +754,6 @@
         xyz="5.0638E-06 -0.0012262 0.056857"
         rpy="0 0 0" />
-      <mass
-        value="0.03" />
+       <mass
+        value="0.001" />
       <inertia
         ixx="0.00014092"
@@ -814,5 +814,5 @@
         rpy="0 0 0" />
       <mass
-        value="0.03" />
+        value="0.001" />
       <inertia
         ixx="0.00018198"
@@ -873,5 +873,5 @@
         rpy="0 0 0" />
       <mass
-        value="0.03" />
+        value="0.001" />
       <inertia
         ixx="4.4099E-05"
@@ -937,6 +937,6 @@
         xyz="5.5511E-17 0.015598 0.034754"
         rpy="0 0 0" />
-      <mass
-        value="0.01" />
+       <mass
+        value="0.001" />
       <inertia
         ixx="1.4683E-05"
@@ -997,5 +997,5 @@
         rpy="0 0 0" />
       <mass
-        value="0.01" />
+        value="0.001" />
       <inertia
         ixx="1.4683E-05"

Commit message: try 2: fixing weird simulation behaviour

File: armadillo_description/urdf/armadillo.xacro (robot description, xacro)
@@ -16,12 +16,12 @@
         xyz="-0.012353 0.000122 0.17716"
         rpy="0 0 0" />
-       <mass value="100.0"/>
+       <mass value="50.0"/>
        <inertia
         ixx="0.31639"
         ixy="-9.1727E-05"
         ixz="-0.093044"
-        iyy="0.17997"
+        iyy="0.0000010997"
         iyz="5.3231E-05"
-        izz="0.16693" />
+        izz="0.000010693" />
     </inertial>
     <visual>
@@ -49,24 +49,4 @@
           </collision>
   </link>
-    <joint name="caster_front_left_joint" type="fixed">
-      <parent link="base_link"/>
-      <child link="caster_front_left_link"/>
-      <origin xyz="0.2 0.24 ${-WHEEL_RADIUS+0.0115+0.05+0.015}" rpy="${-M_PI/2} 0 0"/>
-    </joint>
-    <link name="caster_front_left_link">
-      <collision>
-        <geometry>
-          <cylinder length="0.0176" radius="0.05"/>
-        </geometry>
-        <origin rpy="0 0 0" xyz="0 0 0"/>
-      </collision>
-      <inertial>
-        <mass value="0.01" />
-        <origin xyz="0 0 0" />
-        <inertia ixx="0.001" ixy="0.0" ixz="0.0"
-                 iyy="0.001" iyz="0.0"
-                 izz="0.001" />
-      </inertial>
-    </link>
     <joint name="caster_back_left_joint" type="fixed">
       <parent link="base_link"/>
@@ -80,24 +60,4 @@
         </geometry>
         <origin rpy="0 0 0" xyz="0 0 -0.03"/>
-      </collision>
-      <inertial>
-        <mass value="0.01" />
-        <origin xyz="0 0 0" />
-        <inertia ixx="0.001" ixy="0.0" ixz="0.0"
-                 iyy="0.001" iyz="0.0"
-                 izz="0.001" />
-      </inertial>
-    </link>
-        <joint name="caster_front_right_joint" type="fixed">
-      <parent link="base_link"/>
-      <child link="caster_front_right_link"/>
-      <origin xyz="0.2 -0.24 ${-WHEEL_RADIUS+0.0115+0.05+0.015}" rpy="${-M_PI/2} 0 0"/>
-    </joint>
-    <link name="caster_front_right_link">
-      <collision>
-        <geometry>
-          <cylinder length="0.0176" radius="0.05"/>
-        </geometry>
-        <origin rpy="0 0 0" xyz="0 0 0"/>
       </collision>
       <inertial>
@@ -136,12 +96,12 @@
         rpy="0 0 0" />
    <mass
-        value="1.8524" />
+        value="0.2024" />
       <inertia
         ixx="0.0069046"
         ixy="-3.8717E-08"
         ixz="2.0707E-07"
-        iyy="0.013153"
+        iyy="0.0013153"
         iyz="-1.0124E-07"
-        izz="0.0069054" />
+        izz="0.1069054" />
       </inertial>
     <visual>
@@ -191,12 +151,12 @@
         rpy="0 0 0" />
         <mass
-        value="1.8524" />
+        value="0.2024" />
       <inertia
         ixx="0.0069046"
         ixy="-3.8717E-08"
         ixz="-2.0707E-07"
-        iyy="0.013153"
+        iyy="0.0013153"
         iyz="1.0124E-07"
-        izz="0.0069054" />
+        izz="0.1069054" />
     </inertial>
     <visual>
@@ -336,12 +296,12 @@
         rpy="0 0 0" />
      <mass
-        value="0.001" />
+        value="0.01" />
       <inertia
         ixx="0.09579"
         ixy="2.4285E-05"
         ixz="-0.0045097"
-        iyy="0.06807"
+        iyy="0.0006807"
         iyz="-7.4938E-05"
-        izz="0.072852" />
+        izz="0.00072852" />
     </inertial>
     <visual>
@@ -373,5 +333,5 @@
         rpy="0 0 0" />
       <geometry>
-        <box size="0.09 0.5 0.8"/>
+        <box size="0.09 0.5 0.6"/>
       </geometry>
     </collision>
@@ -403,5 +363,5 @@
         rpy="0 0 0" />
       <mass
-        value="0.001" />
+        value="0.01" />
       <inertia
         ixx="3.6365E-05"
@@ -462,5 +422,5 @@
         rpy="0 0 0" />
       <mass
-        value="0.001" />
+        value="0.01" />
       <inertia
         ixx="0.00056403"
@@ -521,5 +481,5 @@
         rpy="0 0 0" />
       <mass
-        value="0.001" />
+        value="0.1" />
       <inertia
         ixx="0.00056403"
@@ -578,5 +538,5 @@
         rpy="0 0 0" />
       <mass
-        value="0.001" />
+        value="0.1" />
       <inertia
         ixx="0.0043595"
@@ -637,5 +597,5 @@
         rpy="0 0 0" />
       <mass
-        value="0.001" />
+        value="0.1" />
       <inertia
         ixx="0.0043595"
@@ -696,5 +656,5 @@
         rpy="0 0 0" />
       <mass
-        value="0.001" />
+        value="0.1" />
       <inertia
         ixx="0.00093237"
@@ -755,5 +715,5 @@
         rpy="0 0 0" />
        <mass
-        value="0.001" />
+        value="0.1" />
       <inertia
         ixx="0.00014092"
@@ -814,5 +774,5 @@
         rpy="0 0 0" />
       <mass
-        value="0.001" />
+        value="0.1" />
       <inertia
         ixx="0.00018198"
@@ -873,5 +833,5 @@
         rpy="0 0 0" />
       <mass
-        value="0.001" />
+        value="0.1" />
       <inertia
         ixx="4.4099E-05"
@@ -938,5 +898,5 @@
         rpy="0 0 0" />
        <mass
-        value="0.001" />
+        value="0.1" />
       <inertia
         ixx="1.4683E-05"
@@ -997,5 +957,5 @@
         rpy="0 0 0" />
       <mass
-        value="0.001" />
+        value="0.1" />
       <inertia
         ixx="1.4683E-05"
