Commit message: try 4: fix gazebo weird behavoiur

File: armadillo_description/urdf/armadillo2_gazebo.xacro (robot description, xacro)
@@ -163,6 +163,6 @@
         </actuator>
     </transmission>
-    <xacro:property name="mu1" value="2.0" />
-    <xacro:property name="mu2" value="2.0" />
+    <xacro:property name="mu1" value="1.5" />
+    <xacro:property name="mu2" value="1.5" />
     <gazebo reference="left_wheel_link">
         <!-- kp and kd for rubber -->
