Commit message: try 3: fix gazebo weird behavoiur

File: armadillo_description/urdf/armadillo2.xacro (robot description, xacro)
@@ -2,5 +2,5 @@
 <robot xmlns:xacro="http://www.ros.org/wiki/xacro" name="armadillo_robot" description="armadillo robot">
  <xacro:property name="M_PI" value="3.1415926535897931" />
- <xacro:property name="WHEEL_RADIUS" value="0.095" />
+ <xacro:property name="WHEEL_RADIUS" value="0.1016" />
  <xacro:include filename="$(find armadillo_description)/urdf/intel_d435.urdf"/>
 <link name="base_footprint"/>
@@ -16,13 +16,14 @@
         xyz="-0.012353 0.000122 0.17716"
         rpy="0 0 0" />
-       <mass value="50.0"/>
-       <inertia
-        ixx="0.31639"
-        ixy="-9.1727E-05"
-        ixz="-0.093044"
-        iyy="0.0000010997"
-        iyz="5.3231E-05"
-        izz="0.000010693" />
-    </inertial>
+       <mass
+        value="5" />
+        <inertia
+          ixx="0.31639"
+          ixy="-9.1727E-05"
+          ixz="-0.093044"
+          iyy="0.017997"
+          iyz="5.3231E-05"
+          izz="0.16693" />
+        </inertial>
     <visual>
       <origin
@@ -95,13 +96,13 @@
         xyz="9.16610941069373E-06 4.59070539915452E-09 8.0609835912647E-06"
         rpy="0 0 0" />
-   <mass
-        value="0.2024" />
+    <mass
+        value="1.8524" />
       <inertia
         ixx="0.0069046"
         ixy="-3.8717E-08"
         ixz="2.0707E-07"
-        iyy="0.0013153"
+        iyy="0.013153"
         iyz="-1.0124E-07"
-        izz="0.1069054" />
+        izz="0.0069054" />
       </inertial>
     <visual>
@@ -150,13 +151,13 @@
         xyz="9.16610941069373E-06 -4.99540929455033E-06 8.06098359126817E-06"
         rpy="0 0 0" />
-        <mass
-        value="0.2024" />
+       <mass
+        value="1.8524" />
       <inertia
         ixx="0.0069046"
         ixy="-3.8717E-08"
         ixz="-2.0707E-07"
-        iyy="0.0013153"
+        iyy="0.013153"
         iyz="1.0124E-07"
-        izz="0.1069054" />
+        izz="0.0069054" />
     </inertial>
     <visual>
@@ -296,12 +297,12 @@
         rpy="0 0 0" />
      <mass
-        value="0.01" />
+        value="0.001" />
       <inertia
         ixx="0.09579"
         ixy="2.4285E-05"
         ixz="-0.0045097"
-        iyy="0.0006807"
+        iyy="0.06807"
         iyz="-7.4938E-05"
-        izz="0.00072852" />
+        izz="0.072852" />
     </inertial>
     <visual>
@@ -333,5 +334,5 @@
         rpy="0 0 0" />
       <geometry>
-        <box size="0.09 0.5 0.6"/>
+        <box size="0.09 0.5 0.8"/>
       </geometry>
     </collision>
@@ -363,5 +364,5 @@
         rpy="0 0 0" />
       <mass
-        value="0.01" />
+        value="0.001" />
       <inertia
         ixx="3.6365E-05"
@@ -422,5 +423,5 @@
         rpy="0 0 0" />
       <mass
-        value="0.01" />
+        value="0.001" />
       <inertia
         ixx="0.00056403"
@@ -481,5 +482,5 @@
         rpy="0 0 0" />
       <mass
-        value="0.1" />
+        value="0.001" />
       <inertia
         ixx="0.00056403"
@@ -538,12 +539,12 @@
         rpy="0 0 0" />
       <mass
-        value="0.1" />
-      <inertia
-        ixx="0.0043595"
-        ixy="-3.1405E-06"
-        ixz="0.00053636"
-        iyy="0.0041046"
-        iyz="-5.2275E-05"
-        izz="0.00081871" />
+        value="0.001" />
+      <inertia
+        ixx="0.00055596"
+        ixy="9.2522E-12"
+        ixz="9.2226E-12"
+        iyy="0.00016945"
+        iyz="6.1918E-06"
+        izz="0.00055286" />
     </inertial>
     <visual>
@@ -597,5 +598,5 @@
         rpy="0 0 0" />
       <mass
-        value="0.1" />
+        value="0.001" />
       <inertia
         ixx="0.0043595"
@@ -656,5 +657,5 @@
         rpy="0 0 0" />
       <mass
-        value="0.1" />
+        value="0.001" />
       <inertia
         ixx="0.00093237"
@@ -714,6 +715,6 @@
         xyz="5.0638E-06 -0.0012262 0.056857"
         rpy="0 0 0" />
-       <mass
-        value="0.1" />
+      <mass
+        value="0.001" />
       <inertia
         ixx="0.00014092"
@@ -774,5 +775,5 @@
         rpy="0 0 0" />
       <mass
-        value="0.1" />
+        value="0.001" />
       <inertia
         ixx="0.00018198"
@@ -833,5 +834,5 @@
         rpy="0 0 0" />
       <mass
-        value="0.1" />
+        value="0.001" />
       <inertia
         ixx="4.4099E-05"
@@ -897,6 +898,6 @@
         xyz="5.5511E-17 0.015598 0.034754"
         rpy="0 0 0" />
-       <mass
-        value="0.1" />
+      <mass
+        value="0.001" />
       <inertia
         ixx="1.4683E-05"
@@ -957,5 +958,5 @@
         rpy="0 0 0" />
       <mass
-        value="0.1" />
+        value="0.001" />
       <inertia
         ixx="1.4683E-05"
@@ -1009,57 +1010,4 @@
 <dynamics damping="0.5" friction="0.5"/>
   </joint>
- <!-- <joint
-    name="intel_d435_joint"
-    type="fixed">
-    <origin
-      xyz="0 0.0143 -0.049"
-      rpy="-3.1416 0 1.5708" />
-    <parent
-      link="wrist_link" />
-    <child
-      link="intel_d435_link" />
-    <axis
-      xyz="0 0 0" />
-    </joint>-->
-  <!--<link
-    name="intel_d435_link">
-    <inertial>
-      <origin
-        xyz="0.00209672590490473 0.00107373429916791 -0.0124264025663287"
-        rpy="0 0 0" />
-      <mass
-        value="0.0446256012085417" />
-      <inertia
-        ixx="2.62358816469287E-05"
-        ixy="3.51148589025883E-07"
-        ixz="3.91275343984781E-11"
-        iyy="4.02618646244092E-06"
-        iyz="-6.05255657169474E-09"
-        izz="2.64982132448102E-05" />
-    </inertial>
-    <visual>
-      <origin
-        xyz="0 0 0.0125"
-        rpy="0 0 0" />
-      <geometry>
-        <mesh
-          filename="package://armadillo_description/mesh/intel_d435.STL" />
-      </geometry>
-      <material
-        name="">
-        <color
-          rgba="0.792156862745098 0.819607843137255 0.933333333333333 1" />
-      </material>
-    </visual>
-    <collision>
-      <origin
-        xyz="0 0 0"
-        rpy="0 0 0" />
-      <geometry>
-        <mesh
-          filename="package://armadillo_description/mesh/intel_d435.STL" />
-      </geometry>
-    </collision>
-  </link>-->
     <joint
     name="intel_d435_joint"

File: armadillo_description/urdf/armadillo2_gazebo.xacro (robot description, xacro)
@@ -1,6 +1,5 @@
 <?xml version="1.0"?>
 <robot xmlns:xacro="http://www.ros.org/wiki/xacro" name="armadillo_robot" description="armadillo robot">
-    <xacro:include filename="$(find armadillo_description)/urdf/armadillo.xacro" />
-    <xacro:include filename="$(find armadillo_gazebo)/macros/intel_cam.xacro" />
+    <xacro:include filename="$(find armadillo_description)/urdf/armadillo2.xacro" />
     <xacro:arg name="kinect2" default="true"/>
     <xacro:arg name="kinect2_hz" default="30.0"/>
@@ -15,6 +14,21 @@
     <!-- intel_cam -->
     <xacro:if value="$(arg intel_cam)">
-        <xacro:include filename="$(find armadillo_gazebo)/macros/intel_cam.xacro" />
-        <xacro:intel_d435_gazebo name="camera" ros_topic="intel_cam"/>
+        <xacro:include filename="$(find armadillo_gazebo)/macros/depth_cam.xacro" />
+        <xacro:DepthCam name="intel_cam"
+                        link="camera_link"
+                        optical_frame="camera_depth_optical_frame"
+                        horizontal_fov="1.592"
+                        img_width="1280"
+                        img_height="800"
+                        img_format="B8G8R8"
+                        clip_near="0.1"
+                        clip_far="100"
+                        update_rate="10.0"
+                        image_topic="color/image_raw"
+                        depth_topic="depth/color/image_raw"
+                        cloud_topic="depth/color/points"
+                        info_topic="color/camera_info"
+                        depth_info_topic="depth/camera_info"
+                        pointcloud_cuttoff="0.2" />
     </xacro:if>
     <!-- kinect 2 -->
@@ -29,10 +43,20 @@
     <xacro:if value="$(arg urf)">
         <xacro:include filename="$(find armadillo_gazebo)/macros/urf.xacro" />
-        <xacro:urf name="front" link="front_urf_link" topic="URF/front" fov="${10.0*M_PI/180.0}" min="0.2" max="5.0"/>
+        <xacro:urf name="front" link="front_urf_link" topic="urf/front" fov="${10.0*M_PI/180.0}" min="0.3" max="5.0" update_rate="10"/>
     </xacro:if>
     <!-- hokuyo  utm-30lx -->
     <xacro:if value="$(arg lidar)">
-        <xacro:include filename="$(find armadillo_gazebo)/macros/hokuyo.xacro" />
-        <xacro:lidar link="laser_link" topic="scan" samples="720" resolution="1" min_angle="-1.5707963" max_angle="1.5707963" range_min="0.1" range_max="30" range_resolution="0.03" />
+        <xacro:include filename="$(find armadillo_gazebo)/macros/lidar.xacro" />
+        <xacro:lidar name="lidar"
+                     link="laser_link"
+                     topic="scan"
+                     update_rate="10"
+                     samples="720"
+                     resolution="1"
+                     min_angle="-1.5707"
+                     max_angle="1.5707"
+                     range_min="0.1"
+                     range_max="30.0"
+                     range_resolution="0.01" />
     </xacro:if>
     <!-- GPS   -->
@@ -75,5 +99,5 @@
         <fdir1>0 0 1</fdir1>
         <maxVel>1.0</maxVel>
-        <minDepth>0.001</minDepth>
+        <minDepth>0.00</minDepth>
     </gazebo>
     <gazebo reference="left_finger_joint">
@@ -88,5 +112,5 @@
         <fdir1>0 0 1</fdir1>
         <maxVel>1.0</maxVel>
-        <minDepth>0.001</minDepth>
+        <minDepth>0.00</minDepth>
     </gazebo>
     <gazebo reference="right_finger_joint">
@@ -139,55 +163,52 @@
         </actuator>
     </transmission>
+    <xacro:property name="mu1" value="2.0" />
+    <xacro:property name="mu2" value="2.0" />
     <gazebo reference="left_wheel_link">
-        <mu1>3.0</mu1>
-        <mu2>3.0</mu2>
-        <kp>1000000.0</kp>
-        <kd>100.0</kd>
-        <minDepth>0.001</minDepth>
-        <maxVel>1.0</maxVel>
+        <!-- kp and kd for rubber -->
+        <kp>1000000.0</kp>
+        <kd>100.0</kd>
+        <mu1>${mu1}</mu1>
+        <mu2>${mu2}</mu2>
+        <fdir1>1 0 0</fdir1>
+        <maxVel>1.0</maxVel>
+        <minDepth>0.00</minDepth>
+        <material>Gazebo/DarkGrey</material>
     </gazebo>
     <gazebo reference="right_wheel_link">
-        <mu1>3.0</mu1>
-        <mu2>3.0</mu2>
-        <kp>1000000.0</kp>
-        <kd>100.0</kd>
-        <minDepth>0.001</minDepth>
-        <maxVel>1.0</maxVel>
-    </gazebo>
-    <gazebo reference="caster_front_right_link">
+        <!-- kp and kd for rubber -->
+        <kp>1000000.0</kp>
+        <kd>100.0</kd>
+        <mu1>${mu1}</mu1>
+        <mu2>${mu2}</mu2>
+        <fdir1>1 0 0</fdir1>
+        <maxVel>1.0</maxVel>
+        <minDepth>0.00</minDepth>
+        <material>Gazebo/DarkGrey</material>
+    </gazebo>
+    <gazebo reference="caster_back_left_link">
+        <!-- kp and kd for rubber -->
+        <kp>1000000.0</kp>
+        <kd>100.0</kd>
         <mu1>0.0</mu1>
         <mu2>0.0</mu2>
-        <kp>1000000.0</kp>
-        <kd>100.0</kd>
-        <minDepth>0.001</minDepth>
-        <maxVel>1.0</maxVel>
+        <fdir1>1 0 0</fdir1>
+        <maxVel>1.0</maxVel>
+        <minDepth>0.00</minDepth>
+        <material>Gazebo/DarkGrey</material>
     </gazebo>
     <gazebo reference="caster_back_right_link">
+    <!-- kp and kd for rubber -->
+        <kp>1000000.0</kp>
+        <kd>100.0</kd>
         <mu1>0.0</mu1>
         <mu2>0.0</mu2>
-        <kp>1000000.0</kp>
-        <kd>100.0</kd>
-        <minDepth>0.001</minDepth>
-        <maxVel>1.0</maxVel>
-    </gazebo>
-        <gazebo reference="caster_front_left_link">
-        <mu1>0.0</mu1>
-        <mu2>0.0</mu2>
-        <kp>1000000.0</kp>
-        <kd>100.0</kd>
-        <minDepth>0.001</minDepth>
-        <maxVel>1.0</maxVel>
-    </gazebo>
-    <gazebo reference="caster_back_left_link">
-        <mu1>0.0</mu1>
-        <mu2>0.0</mu2>
-        <kp>1000000.0</kp>
-        <kd>100.0</kd>
-        <minDepth>0.001</minDepth>
-        <maxVel>1.0</maxVel>
+        <fdir1>1 0 0</fdir1>
+        <maxVel>1.0</maxVel>
+        <minDepth>0.00</minDepth>
+        <material>Gazebo/DarkGrey</material>
     </gazebo>
     <gazebo reference="base_link">
-        <mu1>0.3</mu1>
-        <mu2>0.3</mu2>
+        <material>Gazebo/Grey</material>
     </gazebo>
     <transmission name="rotation1_joint_trans">

File: armadillo_gazebo/macros/cam.xacro (robot description, xacro)
@@ -1,9 +1,20 @@
+<?xml version="1.0"?>
 <robot xmlns:xacro="http://www.ros.org/wiki/xacro" name="Camera" description="Camera sensor">
-	<xacro:macro name="Camera" params="name link image_width image_height image_format clip_near clip_far">
+	<xacro:macro name="Camera" params="name
+              link
+              image_width
+              image_height
+              image_format
+              clip_near
+              clip_far
+              image_topic
+              info_topic
+              update_rate
+              horizontal_fov">
 		<gazebo reference="${link}">
 			<sensor type="camera" name="${name}">
-				<update_rate>30.0</update_rate>
+				<update_rate>${update_rate}</update_rate>
 				<camera name="${name}">
-					<horizontal_fov>1.3962634</horizontal_fov>
+					<horizontal_fov>${horizontal_fov}</horizontal_fov>
 					<image>
 						<width>${image_width}</width>
@@ -25,6 +36,6 @@
 					<updateRate>0.0</updateRate>
 					<cameraName>${name}</cameraName>
-					<imageTopicName>image_raw</imageTopicName>
-					<cameraInfoTopicName>camera_info</cameraInfoTopicName>
+					<imageTopicName>${image_topic}</imageTopicName>
+					<cameraInfoTopicName>${info_topic}</cameraInfoTopicName>
 					<frameName>${link}</frameName>
 					<hackBaseline>0.07</hackBaseline>

File: armadillo_gazebo/macros/imu.xacro (robot description, xacro)
@@ -1,24 +1,35 @@
 <?xml version="1.0"?>
 <robot xmlns:xacro="http://www.ros.org/wiki/xacro" name="IMU" description="IMU sensor">
-	<xacro:macro name="imu" params="link hz topic">
- <gazebo reference="${link}">
-    <gravity>true</gravity>
-    <sensor name="imu_sensor" type="imu">
-      <always_on>true</always_on>
-      <update_rate>${hz}</update_rate>
-      <visualize>false</visualize>
-      <topic>__default_topic__</topic>
-      <plugin filename="libgazebo_ros_imu_sensor.so" name="imu_plugin">
-        <topicName>${topic}</topicName>
-        <bodyName>${link}</bodyName>
-        <updateRateHZ>${hz}</updateRateHZ>
-        <gaussianNoise>0.01</gaussianNoise>
-        <xyzOffset>0 0 0</xyzOffset>
-        <rpyOffset>0 0 0</rpyOffset>
-        <frameName>${link}</frameName>
-      </plugin>
-      <pose>0 0 0 0 0 0</pose>
-    </sensor>
-  </gazebo>
-	</xacro:macro>
+ <xacro:macro name="imu" params="link hz topic">
+    <gazebo reference="${link}">
+        <gravity>true</gravity>
+        <sensor name="imu_sensor" type="imu">
+        <always_on>true</always_on>
+        <update_rate>${hz}</update_rate>
+        <visualize>false</visualize>
+        <topic>${topic}/data</topic>
+        <plugin filename="libgazebo_ros_imu_sensor.so" name="imu_plugin">
+            <topicName>${topic}</topicName>
+            <bodyName>${link}</bodyName>
+            <updateRateHZ>${hz}</updateRateHZ>
+            <gaussianNoise>0.01</gaussianNoise>
+            <xyzOffset>0 0 0</xyzOffset>
+            <rpyOffset>0 0 0</rpyOffset>
+            <frameName>${link}</frameName>
+        </plugin>
+        <pose>0 0 0 0 0 0</pose>
+        </sensor>
+    </gazebo>
+    <gazebo>
+            <plugin name="GazeboRosMagnetic" filename="libhector_gazebo_ros_magnetic.so">
+                    <updateRate>50.0</updateRate>
+                    <bodyName>${link}</bodyName>
+                    <frameId>${link}</frameId>
+                    <topicName>${topic}/magnetic</topicName>
+                    <offset>0 0 0</offset>
+                    <drift>0.0 0.0 0.0</drift>
+                    <gaussianNoise>1.3e-2 1.3e-2 1.3e-2</gaussianNoise>
+            </plugin>
+    </gazebo>
+  </xacro:macro>
 </robot>

Commit message: try 4: fix gazebo weird behavoiur

File: armadillo_description/urdf/armadillo2.xacro (robot description, xacro)
@@ -97,10 +97,10 @@
         rpy="0 0 0" />
     <mass
-        value="0.8524" />
+        value="0.5" />
       <inertia
         ixx="0.0069046"
         ixy="-3.8717E-08"
         ixz="2.0707E-07"
-        iyy="0.013153"
+        iyy="0.01"
         iyz="-1.0124E-07"
         izz="0.0069054" />
@@ -152,10 +152,10 @@
         rpy="0 0 0" />
        <mass
-        value="0.8524" />
+        value="0.5" />
       <inertia
         ixx="0.0069046"
         ixy="-3.8717E-08"
         ixz="-2.0707E-07"
-        iyy="0.013153"
+        iyy="0.01"
         iyz="1.0124E-07"
         izz="0.0069054" />
@@ -202,4 +202,18 @@
  <link
     name="caster_left_link">
+     <inertial>
+      <origin
+        xyz="9.16610941069373E-06 -4.99540929455033E-06 8.06098359126817E-06"
+        rpy="0 0 0" />
+       <mass
+        value="0.1" />
+      <inertia
+        ixx="0.0069046"
+        ixy="-3.8717E-08"
+        ixz="-2.0707E-07"
+        iyy="0.01"
+        iyz="1.0124E-07"
+        izz="0.0069054" />
+    </inertial>
     <visual>
       <origin
@@ -262,4 +276,18 @@
   <link
     name="caster_right_link">
+      <inertial>
+      <origin
+        xyz="9.16610941069373E-06 -4.99540929455033E-06 8.06098359126817E-06"
+        rpy="0 0 0" />
+       <mass
+        value="0.1" />
+      <inertia
+        ixx="0.0069046"
+        ixy="-3.8717E-08"
+        ixz="-2.0707E-07"
+        iyy="0.01"
+        iyz="1.0124E-07"
+        izz="0.0069054" />
+    </inertial>
     <visual>
       <origin

Commit message: try 4: fix gazebo weird behavoiur

File: armadillo_description/urdf/armadillo2.xacro (robot description, xacro)
@@ -17,5 +17,5 @@
         rpy="0 0 0" />
        <mass
-        value="30" />
+        value="100" />
         <inertia
           ixx="0.31639"
@@ -325,12 +325,12 @@
         rpy="0 0 0" />
      <mass
-        value="0.001" />
+        value="0.01" />
       <inertia
         ixx="0.09579"
         ixy="2.4285E-05"
         ixz="-0.0045097"
-        iyy="0.06807"
+        iyy="0.0001"
         iyz="-7.4938E-05"
-        izz="0.072852" />
+        izz="0.00032852" />
     </inertial>
     <visual>
@@ -362,5 +362,5 @@
         rpy="0 0 0" />
       <geometry>
-        <box size="0.09 0.5 0.8"/>
+        <box size="0.09 0.5 0.6"/>
       </geometry>
     </collision>
@@ -383,5 +383,5 @@
       effort="0.001"
       velocity="0.1" />
-<dynamics damping="0.1" friction="0"/>
+<!--<dynamics damping="0.1" friction="0"/>-->
   </joint>
   <link
@@ -442,5 +442,5 @@
       effort="0.5"
       velocity="2" />
-<dynamics damping="0.1" friction="0"/>
+<!--<dynamics damping="0.1" friction="0"/>-->
   </joint>
   <link
@@ -501,5 +501,5 @@
       effort="0.5"
       velocity="2" />
-<dynamics damping="0.1" friction="0"/>
+<!--<dynamics damping="0.1" friction="0"/>-->
   </joint>
   <link
@@ -617,5 +617,5 @@
       upper="1.57"
       velocity="2.0" />
-<dynamics damping="0.1" friction="0"/>
+<!--<dynamics damping="0.1" friction="0"/>-->
   </joint>
   <link
@@ -676,5 +676,5 @@
       upper="1.95"
       velocity="2.0" />
-<dynamics damping="0.1" friction="0"/>
+<!--<dynamics damping="0.1" friction="0"/>-->
   </joint>
   <link
@@ -735,5 +735,5 @@
       upper="2.3522"
       velocity="2.0" />
-<dynamics damping="0.1" friction="0"/>
+<!--<dynamics damping="0.1" friction="0"/>-->
   </joint>
   <link
@@ -794,5 +794,5 @@
       upper="1.57"
       velocity="2.0" />
-<dynamics damping="0.1" friction="0"/>
+<!--<dynamics damping="0.1" friction="0"/>-->
   </joint>
   <link
@@ -853,5 +853,5 @@
       upper="1.57"
       velocity="2.0" />
-<dynamics damping="0.1" friction="0"/>
+<!--<dynamics damping="0.1" friction="0"/>-->
   </joint>
   <link
@@ -912,5 +912,5 @@
       upper="3.14"
       velocity="2.0" />
-<dynamics damping="0.5" friction="0.5"/>
+<!--<dynamics damping="0.5" friction="0.5"/>-->
   </joint>
   <link name="gripper_link"/>
@@ -977,5 +977,5 @@
       upper="1.57"
       velocity="0.1" />
-<dynamics damping="0.5" friction="0.5"/>
+<!--<dynamics damping="0.5" friction="0.5"/>-->
   </joint>
   <link
@@ -1036,5 +1036,5 @@
       upper="1.57"
       velocity="0.1" />
-<dynamics damping="0.5" friction="0.5"/>
+<!--<dynamics damping="0.5" friction="0.5"/>-->
   </joint>
     <joint

Commit message: try 4: fix gazebo weird behavoiur

File: armadillo_description/urdf/armadillo2.xacro (robot description, xacro)
@@ -17,5 +17,5 @@
         rpy="0 0 0" />
        <mass
-        value="100" />
+        value="50" />
         <inertia
           ixx="0.31639"
@@ -65,7 +65,11 @@
         <mass value="0.01" />
         <origin xyz="0 0 0" />
-        <inertia ixx="0.001" ixy="0.0" ixz="0.0"
-                 iyy="0.001" iyz="0.0"
-                 izz="0.001" />
+        <inertia
+        ixx="0.0069046"
+        ixy="-3.8717E-08"
+        ixz="2.0707E-07"
+        iyy="0.01"
+        iyz="-1.0124E-07"
+        izz="0.0069054" />
       </inertial>
     </link>
@@ -85,18 +89,5 @@
         <mass value="0.01" />
         <origin xyz="0 0 0" />
-        <inertia ixx="0.001" ixy="0.0" ixz="0.0"
-                 iyy="0.001" iyz="0.0"
-                 izz="0.001" />
-      </inertial>
-    </link>
- <link
-    name="left_wheel_link">
-    <inertial>
-      <origin
-        xyz="9.16610941069373E-06 4.59070539915452E-09 8.0609835912647E-06"
-        rpy="0 0 0" />
-    <mass
-        value="0.5" />
-      <inertia
+        <inertia
         ixx="0.0069046"
         ixy="-3.8717E-08"
@@ -106,4 +97,21 @@
         izz="0.0069054" />
       </inertial>
+    </link>
+ <link
+    name="left_wheel_link">
+    <inertial>
+      <origin
+        xyz="9.16610941069373E-06 4.59070539915452E-09 8.0609835912647E-06"
+        rpy="0 0 0" />
+    <mass
+        value="1.5" />
+      <inertia
+        ixx="0.0069046"
+        ixy="-3.8717E-08"
+        ixz="2.0707E-07"
+        iyy="0.01"
+        iyz="-1.0124E-07"
+        izz="0.0069054" />
+      </inertial>
     <visual>
       <origin
@@ -152,5 +160,5 @@
         rpy="0 0 0" />
        <mass
-        value="0.5" />
+        value="1.5" />
       <inertia
         ixx="0.0069046"
@@ -325,5 +333,5 @@
         rpy="0 0 0" />
      <mass
-        value="0.01" />
+        value="0.001" />
       <inertia
         ixx="0.09579"

File: armadillo_description/urdf/armadillo2_gazebo.xacro (robot description, xacro)
@@ -163,6 +163,6 @@
         </actuator>
     </transmission>
-    <xacro:property name="mu1" value="1.5" />
-    <xacro:property name="mu2" value="1.5" />
+    <xacro:property name="mu1" value="0.5" />
+    <xacro:property name="mu2" value="0.5" />
     <gazebo reference="left_wheel_link">
         <!-- kp and kd for rubber -->
