Commit message: stablizing urdf model

File: armadillo_description/urdf/armadillo2.xacro (robot description, xacro)
@@ -17,12 +17,12 @@
         rpy="0 0 0" />
        <mass
-        value="50" />
+        value="30" />
         <inertia
-          ixx="0.31639"
+          ixx="0.61639"
           ixy="-9.1727E-05"
           ixz="-0.093044"
-          iyy="0.017997"
+          iyy="0.57997"
           iyz="5.3231E-05"
-          izz="0.16693" />
+          izz="0.36693" />
         </inertial>
     <visual>
@@ -63,5 +63,5 @@
       </collision>
       <inertial>
-        <mass value="0.01" />
+        <mass value="0.0001" />
         <origin xyz="0 0 0" />
         <inertia
@@ -87,5 +87,5 @@
       </collision>
       <inertial>
-        <mass value="0.01" />
+        <mass value="0.0001" />
         <origin xyz="0 0 0" />
         <inertia
@@ -215,5 +215,5 @@
         rpy="0 0 0" />
        <mass
-        value="1.1" />
+        value="0.0001" />
       <inertia
         ixx="0.0069046"
@@ -289,5 +289,5 @@
         rpy="0 0 0" />
        <mass
-        value="1.1" />
+        value="0.0001" />
       <inertia
         ixx="0.0069046"
@@ -333,6 +333,13 @@
         rpy="0 0 0" />
      <mass
-        value="0.001" />
-      <inertia
+         value="0.035511" />
+     <inertia
+        ixx="0.19579"
+        ixy="2.4285E-05"
+        ixz="-0.0045097"
+        iyy="0.16807"
+        iyz="-7.4938E-05"
+        izz="0.072852" />
+    <!--  <inertia
         ixx="0.09579"
         ixy="2.4285E-05"
@@ -340,5 +347,5 @@
         iyy="0.0001"
         iyz="-7.4938E-05"
-        izz="0.00032852" />
+        izz="0.00032852" />-->
     </inertial>
     <visual>
